Commit message: Constructor with randomness done and new limbs to see differences

File: URDFs_set/body_Link_amarelo.urdf (robot description, URDF)
Before this commit: robot L_WHEEL, 2 links, 1 joints
Links:
- removed link link_Helper
- removed link wheel_link
- added link body_joint_link, mass 0.5; collision sphere radius=0.05; visual sphere length=0.07 radius=0.02
- added link body_link, mass 5.0; collision cylinder length=0.1875 radius=0.05625; visual cylinder length=0.1875 radius=0.05625
Joints:
- removed joint wheel_back_joint
- added joint top_sphere_joint_body: type fixed, parent body_link, child body_joint_link, origin xyz=0 0 0.0875 rpy=1.5 0 0

File: URDFs_set/body_Link_verde.urdf (robot description, URDF)
Before this commit: robot L_WHEEL, 2 links, 1 joints
Links:
- removed link link_Helper
- removed link wheel_link
- added link body_joint_link, mass 0.5; collision sphere radius=0.05; visual sphere length=0.07 radius=0.02
- added link body_link, mass 5.0; collision cylinder length=0.1875 radius=0.05625; visual cylinder length=0.1875 radius=0.05625
Joints:
- removed joint wheel_back_joint
- added joint top_sphere_joint_body: type fixed, parent body_link, child body_joint_link, origin xyz=0 0 0.0875 rpy=1.5 0 0

File: URDFs_set/limb_Link_amarelo.urdf (robot description, URDF)
Before this commit: robot Link:small, 2 links, 1 joints
Links:
- removed link limb_small_link_robot
- added link limb_joint_bottom_blue_link, mass 2.5; collision sphere radius=0.03125; visual sphere radius=0.03125
- link limb_link: geometry collision cylinder length=0.1875 radius=0.03125; visual cylinder length=0.1875 radius=0.03125
Joints:
- joint bot_sphere_joint_limb: origin xyz=0 0 0.05 rpy=0 0 0 -> xyz=0 0 0.09 rpy=0 0 0; parent limb_small_link_robot -> limb_joint_bottom_blue_link

File: URDFs_set/limb_Link_preto.urdf (robot description, URDF)
Before this commit: robot Link:small, 2 links, 1 joints
Links:
- removed link limb_small_link_robot
- added link limb_joint_bottom_blue_link, mass 2.5; collision sphere radius=0.03125; visual sphere radius=0.03125
- link limb_link: geometry collision cylinder length=0.1875 radius=0.03125; visual cylinder length=0.1875 radius=0.03125
Joints:
- joint bot_sphere_joint_limb: origin xyz=0 0 0.05 rpy=0 0 0 -> xyz=0 0 0.09 rpy=0 0 0; parent limb_small_link_robot -> limb_joint_bottom_blue_link

File: URDFs_set/limb_Link_rosa.urdf (robot description, URDF)
Before this commit: robot Link:small, 2 links, 1 joints
Links:
- removed link limb_small_link_robot
- added link limb_joint_bottom_blue_link, mass 2.5; collision sphere radius=0.03125; visual sphere radius=0.03125
- link limb_link: geometry collision cylinder length=0.1875 radius=0.03125; visual cylinder length=0.1875 radius=0.03125
Joints:
- joint bot_sphere_joint_limb: origin xyz=0 0 0.05 rpy=0 0 0 -> xyz=0 0 0.09 rpy=0 0 0; parent limb_small_link_robot -> limb_joint_bottom_blue_link

File: URDFs_set/limb_Link_verde.urdf (robot description, URDF)
Before this commit: robot Link:small, 2 links, 1 joints
Links:
- removed link limb_small_link_robot
- added link limb_joint_bottom_blue_link, mass 2.5; collision sphere radius=0.03125; visual sphere radius=0.03125
- link limb_link: geometry collision cylinder length=0.1875 radius=0.03125; visual cylinder length=0.1875 radius=0.03125
Joints:
- joint bot_sphere_joint_limb: origin xyz=0 0 0.05 rpy=0 0 0 -> xyz=0 0 0.09 rpy=0 0 0; parent limb_small_link_robot -> limb_joint_bottom_blue_link

File: URDFs_set/limb_Link_vermelho.urdf (robot description, URDF)
Before this commit: robot Link:small, 2 links, 1 joints
Links:
- removed link limb_small_link_robot
- added link limb_joint_bottom_blue_link, mass 2.5; collision sphere radius=0.03125; visual sphere radius=0.03125
- link limb_link: geometry collision cylinder length=0.1875 radius=0.03125; visual cylinder length=0.1875 radius=0.03125
Joints:
- joint bot_sphere_joint_limb: origin xyz=0 0 0.05 rpy=0 0 0 -> xyz=0 0 0.09 rpy=0 0 0; parent limb_small_link_robot -> limb_joint_bottom_blue_link
