Commit message: New body link

File: URDFs_set/body_Link_HEX.urdf (robot description, URDF)
Before this commit: robot BODY_LINK, 2 links, 1 joints
Links:
- link body_joint_link: geometry collision sphere radius=0.05; visual sphere radius=0.02
- link body_link: geometry collision mesh filename=package://meshes/hexagon.stl; visual mesh filename=package://meshes/hexagon.stl
