Commit message: Links and Joints work on and new Constructor

File: URDFs_set/B_joint_continuous.urdf (robot description, URDF)
Before this commit: robot continuous_joint, 0 links, 1 joints
Links:
- added link auxiliar, mass 0.5; collision sphere radius=0.05; visual cylinder length=0.07 radius=0.05
Joints:
- added joint revolute_joint: type fixed, parent auxiliar, child body_link, origin xyz=0 0 -0.15 rpy=0 0 0
- joint continuous_joint: axis 0 1 0 -> 0 0 1; child bottom_attachment -> auxiliar; parent top_attachment -> body_joint_link

File: URDFs_set/L_joint_continuous.urdf (robot description, URDF)
Before this commit: robot continuous_joint, 0 links, 1 joints
Links:
- added link auxiliar, mass 0.5; collision sphere radius=0.05; visual cylinder length=0.07 radius=0.05
Joints:
- added joint fixed_joint: type fixed, parent auxiliar, child limb_joint_bottom_blue_link, origin xyz=0 0 -0.15 rpy=0 0 0
- joint continuous_joint: axis 0 1 0 -> 0 0 1; child bottom_attachment -> auxiliar; origin xyz=0 0 0 rpy=0 0 0 -> xyz=0 0 0 rpy=1.6 0 0; parent top_attachment -> body_joint_link

File: URDFs_set/limb_Link.urdf (robot description, URDF)
Before this commit: robot Limb_link_robot, 3 links, 2 joints
Links:
- removed link bottom_attachment
- removed link top_attachment
- added link limb_joint_bottom_blue_link, mass 2.5; collision sphere radius=0.03125; visual sphere radius=0.03125
- link limb_link: mass 0.5 -> 2.5; geometry collision cylinder length=0.1875 radius=0.03125; visual cylinder length=0.1875 radius=0.03125
Joints:
- removed joint bottom_joint
- removed joint top_joint
- added joint bot_sphere_joint_limb: type fixed, parent limb_joint_bottom_blue_link, child limb_link, origin xyz=0 0 0.09 rpy=0 0 0

File: URDFs_set/testeURDF.urdf (robot description, URDF)
Before this commit: robot Body_link_robot, 3 links, 2 joints
Links:
- removed link top_attachment
- added link auxiliar, mass 0.5; collision sphere radius=0.05; visual cylinder length=0.07 radius=0.05
- added link body_joint_link, mass 0.5; collision sphere radius=0.05; visual sphere length=0.07 radius=0.02
- added link limb_joint_bottom_blue_link, mass 2.5; collision sphere radius=0.03125; visual sphere radius=0.03125
- link body_link: mass 1.0 -> 5.0; geometry collision cylinder length=0.1875 radius=0.05625; visual cylinder length=0.1875 radius=0.05625
- link limb_link: mass 0.5 -> 2.5; geometry collision cylinder length=0.1875 radius=0.03125; visual cylinder length=0.1875 radius=0.03125
Joints:
- removed joint revolute_joint
- removed joint top_joint
- added joint bot_sphere_joint_limb: type fixed, parent limb_joint_bottom_blue_link, child limb_link, origin xyz=0 0 0.09 rpy=0 0 0
- added joint continuous_joint: type continuous, parent body_joint_link, child auxiliar, origin xyz=0 0 0 rpy=1.6 0 0, axis 0 0 1
- added joint fixed_joint: type fixed, parent auxiliar, child limb_joint_bottom_blue_link, origin xyz=0 0 -0.15 rpy=0 0 0
- added joint top_sphere_joint_body: type fixed, parent body_link, child body_joint_link, origin xyz=0 0 0.0875 rpy=1.5 0 0

Commit message: Rules and update and addiction of links

File: URDFs_set/B_joint_continuous.urdf (robot description, URDF)
Before this commit: robot B_JOINT_CONTI, 1 links, 2 joints
Joints:
- removed joint revolute_joint
- added joint fixed_joint: type fixed, parent auxiliar, child body_link, origin xyz=0 0 -0.15 rpy=0 0 0

File: URDFs_set/L_joint_fixed.urdf (robot description, URDF)
Before this commit: robot L_JOINT_FIX, 1 links, 2 joints
Joints:
- removed joint continuous_joint

File: URDFs_set/L_joint_revolute_horizontal.urdf (robot description, URDF)
Before this commit: robot L_JOINT_CONTI, 1 links, 2 joints
Joints:
- removed joint continuous_joint
- added joint revolute_joint: type revolute, parent body_joint_link, child auxiliar, origin xyz=0 0.04 0 rpy=-1.5 0 0, axis 0 0 1, limit lower=-1.14 upper=1.14 effort=1.0 velocity=1.0
- joint fixed_joint: origin xyz=0 0 -0.15 rpy=0 0 0 -> xyz=0 0.2 0.005 rpy=1.6 0 0

File: URDFs_set/body_Link_CUBE.urdf (robot description, URDF)
Before this commit: robot BODY_LINK, 7 links, 6 joints
Links:
- removed link back_sphere
- removed link bottom_sphere
- removed link front_sphere
- removed link left_sphere
- removed link right_sphere
- removed link top_sphere
Joints:
- removed joint back_sphere_joint_body
- removed joint bottom_sphere_joint_body
- removed joint front_sphere_joint_body
- removed joint left_sphere_joint_body
- removed joint right_sphere_joint_body
- removed joint top_sphere_joint_body

File: URDFs_set/wheel_link.urdf (robot description, URDF)
Before this commit: robot L_WHEEL, 2 links, 1 joints
Links:
- removed link link_Helper
Joints:
- removed joint wheel_back_joint
