Commit message: Teste for autonomous assembly #3
Issue #1 resolvido

File: URDFs_set/B_joint_fixed_BACK.urdf (robot description, URDF)
Before this commit: robot B_JOINT_fixed, 1 links, 1 joints
Joints:
- added joint fixed_joint_: type fixed, parent link_square, child , origin xyz=0 0 0 rpy=0 0 0
- joint fixed_joint: child  -> link_square; origin xyz=0 -0.07 0 rpy=0 0 0 -> xyz=0 0 0 rpy=0 0 0; parent link_square -> 

File: URDFs_set/limb_Link.urdf (robot description, URDF)
Before this commit: robot Limb_LINK, 3 links, 2 joints
Joints:
- joint fixed_joint_: parent aux_sphere -> 
