Commit message: Link color correction for Pybullet, new testing scripts, New Enviroment and PPO Training and testing

File: URDFs_set/limb_Link.urdf (robot description, URDF)
Before this commit: robot Limb_LINK, 3 links, 2 joints
Links:
- link limb_link: geometry collision cylinder length=0.1875 radius=0.03125; visual cylinder length=0.1875 radius=0.03125

File: URDFs_set/limb_Link_Small.urdf (robot description, URDF)
Before this commit: robot Link:small, 3 links, 2 joints
Links:
- link limb_link: geometry collision cylinder length=0.10 radius=0.02125; visual cylinder length=0.10 radius=0.02125

File: URDFs_set/wheel_link.urdf (robot description, URDF)
Before this commit: robot L_WHEEL, 2 links, 1 joints
Links:
- link limb_link: geometry collision cylinder length=0.025 radius=0.07; visual cylinder length=0.025 radius=0.07

File: corrected_robot10.urdf (robot description, URDF)
Before this commit: robot combined_robot0, 16 links, 15 joints
Links:
- removed link 16 L_joint_revolute
- removed link 17 wheel_link
- removed link 3 limb_Link
- removed link 4 L_joint_continuous
- removed link 5 wheel_link
- removed link 7 B_joint_fixed
- removed link 8 body_Link_CUBE
- removed link Sphere_2
- added link 10 wheel_link, mass 0.5; collision cylinder length=0.025 radius=0.07; visual cylinder length=0.025 radius=0.07
- added link 3 limb_Link_Small, mass 2.5; collision cylinder length=0.10 radius=0.02125; visual cylinder length=0.10 radius=0.02125
- added link 4 L_joint_fixed, mass 1.0; collision box size=0.04 0.04 0.04; visual box size=0.04 0.04 0.04
- added link 5 limb_Link_Small, mass 2.5; collision cylinder length=0.10 radius=0.02125; visual cylinder length=0.10 radius=0.02125
- added link 9 L_joint_continuous, mass 0.5; collision cylinder length=0.06 radius=0.04; visual cylinder length=0.06 radius=0.04
- added link extra_sphere_2, mass 2.5; collision sphere radius=0.02125; visual sphere radius=0.02125
- link blackSphere_0: geometry collision sphere radius=0.01; visual sphere radius=0.01
- link blackSphere_1: geometry collision sphere radius=0.01; visual sphere radius=0.01
- link extra_sphere_1: geometry collision sphere radius=0.02125; visual sphere radius=0.02125
Joints:
- removed joint joint_13
- removed joint joint_14
- joint joint_0: origin xyz=0.05 0 0 rpy=0 0 0 -> xyz=0 -0.05 0 rpy=0 0 0
- joint joint_1: origin xyz=0 0 0 rpy=0 1.55 0 -> xyz=0 0 0 rpy=1.55 0 0
- joint joint_10: axis (none) -> 0 0 1; child 8 body_Link_CUBE -> 9 L_joint_continuous; limit (none) -> lower=-1000 upper=1000 effort=1.0 velocity=1.0; origin xyz=0 0.07 0 rpy=0 0 0 -> xyz=0 0 0 rpy=0 0 0; parent 7 B_joint_fixed -> Sphere_1; type fixed -> revolute
- joint joint_11: child Sphere_2 -> blackSphere_2; origin xyz=0 0 -0.05 rpy=0 0 0 -> xyz=0 0 0 rpy=0 0 0; parent 1 body_Link_CUBE -> 9 L_joint_continuous
- joint joint_12: axis 0 0 1 -> (none); child 16 L_joint_revolute -> 10 wheel_link; limit lower=-0.75 upper=0.75 effort=1.0 velocity=1.0 -> (none); origin xyz=0 0 0 rpy=0 -1.55 0 -> xyz=0 0 0.04 rpy=0 0 0; parent Sphere_2 -> blackSphere_2; type revolute -> fixed
- joint joint_3: child 3 limb_Link -> 3 limb_Link_Small; origin xyz=0 0 0.09 rpy=0 0 3.15 -> xyz=0 0 0.045 rpy=0 0 3.15
- joint joint_4: origin xyz=0 0 0.09 rpy=0 0 0 -> xyz=0 0 0.05 rpy=0 0 0; parent 3 limb_Link -> 3 limb_Link_Small
- joint joint_5: axis 0 0 1 -> (none); child 4 L_joint_continuous -> 4 L_joint_fixed; limit lower=-1000 upper=1000 effort=1.0 velocity=1.0 -> (none); type revolute -> fixed
- joint joint_6: parent 4 L_joint_continuous -> 4 L_joint_fixed
- joint joint_7: child 5 wheel_link -> 5 limb_Link_Small; origin xyz=0 0 0.04 rpy=0 0 0 -> xyz=0 0 0.045 rpy=0 0 3.15
- joint joint_8: child Sphere_1 -> extra_sphere_2; origin xyz=0 0.05 0 rpy=0 0 0 -> xyz=0 0 0.05 rpy=0 0 0; parent 1 body_Link_CUBE -> 5 limb_Link_Small
- joint joint_9: child 7 B_joint_fixed -> Sphere_1; origin xyz=0 0 0 rpy=0 0 0 -> xyz=0 0 0.05 rpy=0 0 0; parent Sphere_1 -> 1 body_Link_CUBE

File: corrected_robot4.urdf (robot description, URDF)
Before this commit: robot combined_robot0, 16 links, 15 joints
Links:
- removed link 16 L_joint_revolute
- removed link 17 wheel_link
- removed link 2 L_joint_fixed
- removed link 3 limb_Link
- removed link 4 L_joint_continuous
- removed link 5 wheel_link
- removed link 7 B_joint_fixed
- removed link 8 body_Link_CUBE
- removed link blackSphere_0
- removed link blackSphere_1
- removed link blackSphere_2
- removed link extra_sphere_1
- added link 10 B_joint_revolute, mass 0.5; collision cylinder length=0.07 radius=0.05; visual cylinder length=0.07 radius=0.05
- added link 11 body_Link_CUBE, mass 5.0; collision box size=0.1 0.1 0.1; visual box size=0.1 0.1 0.1
- added link 17 B_joint_fixed, mass 1.0; collision box size=0.07 0.07 0.07; visual box size=0.07 0.07 0.07
- added link 18 body_Link_CUBE, mass 5.0; collision box size=0.1 0.1 0.1; visual box size=0.1 0.1 0.1
- added link 2 B_joint_revolute, mass 0.5; collision cylinder length=0.07 radius=0.05; visual cylinder length=0.07 radius=0.05
- added link 24 B_joint_fixed, mass 1.0; collision box size=0.07 0.07 0.07; visual box size=0.07 0.07 0.07
- added link 25 body_Link_CUBE, mass 5.0; collision box size=0.1 0.1 0.1; visual box size=0.1 0.1 0.1
- added link 3 body_Link_CUBE, mass 5.0; collision box size=0.1 0.1 0.1; visual box size=0.1 0.1 0.1
- added link Sphere_3, mass 0.5; collision sphere radius=0.02; visual sphere radius=0.02
- added link Sphere_4, mass 0.5; collision sphere radius=0.02; visual sphere radius=0.02
- added link Sphere_5, mass 0.5; collision sphere radius=0.02; visual sphere radius=0.02
Joints:
- removed joint joint_14
- joint joint_0: origin xyz=0.05 0 0 rpy=0 0 0 -> xyz=0 -0.05 0 rpy=0 0 0
- joint joint_1: axis (none) -> 0 0 1; child 2 L_joint_fixed -> 2 B_joint_revolute; limit (none) -> lower=-1 upper=1 effort=1.0 velocity=1.0; origin xyz=0 0 0 rpy=0 1.55 0 -> xyz=0 0 0 rpy=0 0 0; type fixed -> revolute
- joint joint_10: child 8 body_Link_CUBE -> 18 body_Link_CUBE; origin xyz=0 0.07 0 rpy=0 0 0 -> xyz=0 0 0.07 rpy=0 0 0; parent 7 B_joint_fixed -> 17 B_joint_fixed
- joint joint_11: child Sphere_2 -> Sphere_5; origin xyz=0 0 -0.05 rpy=0 0 0 -> xyz=0.05 0 0 rpy=0 0 0
- joint joint_12: axis 0 0 1 -> (none); child 16 L_joint_revolute -> 24 B_joint_fixed; limit lower=-0.75 upper=0.75 effort=1.0 velocity=1.0 -> (none); origin xyz=0 0 0 rpy=0 -1.55 0 -> xyz=0 0 0 rpy=0 0 0; parent Sphere_2 -> Sphere_5; type revolute -> fixed
- joint joint_13: child blackSphere_2 -> 25 body_Link_CUBE; origin xyz=0 0 0 rpy=0 -1.6 0 -> xyz=0.07 0 0 rpy=0 0 0; parent 16 L_joint_revolute -> 24 B_joint_fixed
- joint joint_2: child blackSphere_0 -> Sphere_1; origin xyz=0 0 0 rpy=0 0 0 -> xyz=0 -0.05 0 rpy=0 0 0; parent 2 L_joint_fixed -> 2 B_joint_revolute
- joint joint_3: child 3 limb_Link -> 3 body_Link_CUBE; origin xyz=0 0 0.09 rpy=0 0 3.15 -> xyz=0 -0.05 0 rpy=0 0 0; parent blackSphere_0 -> Sphere_1
- joint joint_4: child extra_sphere_1 -> Sphere_2; origin xyz=0 0 0.09 rpy=0 0 0 -> xyz=0 0 -0.05 rpy=0 0 0; parent 3 limb_Link -> 1 body_Link_CUBE
- joint joint_5: child 4 L_joint_continuous -> 10 B_joint_revolute; limit lower=-1000 upper=1000 effort=1.0 velocity=1.0 -> lower=-1 upper=1 effort=1.0 velocity=1.0; origin xyz=0 0 0 rpy=0 0 0 -> xyz=0 0 0 rpy=1.55 0 0; parent extra_sphere_1 -> Sphere_2
- joint joint_6: child blackSphere_1 -> Sphere_3; origin xyz=0 0 0 rpy=0 0 0 -> xyz=0 -0.05 0 rpy=0 0 0; parent 4 L_joint_continuous -> 10 B_joint_revolute
- joint joint_7: child 5 wheel_link -> 11 body_Link_CUBE; origin xyz=0 0 0.04 rpy=0 0 0 -> xyz=0 -0.05 0 rpy=0 0 0; parent blackSphere_1 -> Sphere_3
- joint joint_8: child Sphere_1 -> Sphere_4; origin xyz=0 0.05 0 rpy=0 0 0 -> xyz=0 0 0.05 rpy=0 0 0
- joint joint_9: child 7 B_joint_fixed -> 17 B_joint_fixed; parent Sphere_1 -> Sphere_4
