Commit message: Update joints and new grammar expansion using tree
The usage of tree in the grammar expansion will try to facilitate the future construction of the robot

File: URDFs_set/L_joint_continuous.urdf (robot description, URDF)
Before this commit: robot L_JOINT_CONTI, 1 links, 2 joints
Joints:
- removed joint joint_12
- added joint joint_2: type fixed, parent auxiliar, child , origin xyz=0 0 -0.04 rpy=0 0 0

File: URDFs_set/L_joint_fixed.urdf (robot description, URDF)
Before this commit: robot L_JOINT_FIX, 1 links, 1 joints
Joints:
- added joint joint_2: type fixed, parent , child , origin xyz=0 0.2 0.005 rpy=1.6 0 0
- joint joint_1: child  -> link_square; origin xyz=0 0.2 0.005 rpy=1.6 0 0 -> xyz=0 0 0 rpy=0 0 0

File: URDFs_set/limb_Link_Small.urdf (robot description, URDF)
Before this commit: robot Link:small, 3 links, 2 joints
Joints:
- removed joint bot_sphere_joint_limb
- removed joint fixed_joint
- added joint joint_1: type fixed, parent aux_sphere, child limb_link, origin xyz=0 0 0.045 rpy=0 0 0
- added joint joint_2: type fixed, parent limb_link, child limb_small_link_robot, origin xyz=0 0 0.05 rpy=0 0 0

File: URDFs_set/wheel_link.urdf (robot description, URDF)
Before this commit: robot L_WHEEL, 1 links, 0 joints
Links:
- added link , mass 0.5; collision sphere radius=0.02; visual sphere radius=0.02
Joints:
- added joint joint_1: type fixed, parent , child wheel_link, origin xyz=0 0 0 rpy=0 0 0

Commit message: Update for collision

File: URDFs_set/L_joint_continuous.urdf (robot description, URDF)
Before this commit: robot L_JOINT_CONTI, 1 links, 2 joints
Joints:
- joint joint_2: origin xyz=0 0 0 rpy=0 0 0 -> xyz=0 0 0.02 rpy=0 0 0

File: URDFs_set/L_joint_fixed.urdf (robot description, URDF)
Before this commit: robot L_JOINT_FIX, 1 links, 2 joints
Joints:
- joint joint_2: origin xyz=0 0 0 rpy=0 0 0 -> xyz=0 0 0.02 rpy=0 0 0

File: URDFs_set/limb_Link.urdf (robot description, URDF)
Before this commit: robot Limb_LINK, 3 links, 2 joints
Joints:
- joint joint_1: origin xyz=0 0 0.03 rpy=0 0 3.15 -> xyz=0 0 0.035 rpy=0 0 3.15

File: URDFs_set/limb_Link_Small.urdf (robot description, URDF)
Before this commit: robot Link:small, 3 links, 2 joints
Joints:
- joint joint_1: origin xyz=0 0 0.022 rpy=0 0 3.15 -> xyz=0 0 0.025 rpy=0 0 3.15

File: URDFs_set/wheel_link.urdf (robot description, URDF)
Before this commit: robot L_WHEEL, 2 links, 1 joints
Joints:
- joint joint_1: origin xyz=0 0 0.02 rpy=0 0 0 -> xyz=0 0 0.025 rpy=0 0 0
