Commit message: Update JointS

File: URDFs_set/B_joint_continuous_BACK.urdf (robot description, URDF)
Before this commit: robot L_JOINT_CONTI, 1 links, 2 joints
Links:
- link auxiliar: geometry collision sphere radius=0.05; visual cylinder length=0.07 radius=0.05
Joints:
- removed joint front_sphere_joint
- added joint fixed_joint: type fixed, parent auxiliar, child body_link2, origin xyz=0 0 0.07 rpy=0 0 0
- joint continuous_joint: origin xyz=0 0 0 rpy=0 0 0 -> xyz=0 0 0 rpy=1.55 0 0; parent  -> back_sphere

File: URDFs_set/B_joint_continuous_BOTTOM.urdf (robot description, URDF)
Before this commit: robot B_JOINT_CONTI, 1 links, 2 joints
Joints:
- joint continuous_joint: parent body_joint_link -> back_sphere
- joint fixed_joint: child body_link -> body_link2; origin xyz=0 0 -0.15 rpy=0 0 0 -> xyz=0 0 -0.07 rpy=0 0 0

File: URDFs_set/B_joint_continuous_FRONT.urdf (robot description, URDF)
Before this commit: robot L_JOINT_CONTI, 1 links, 2 joints
Links:
- link auxiliar: geometry collision sphere radius=0.05; visual cylinder length=0.07 radius=0.05
Joints:
- removed joint front_sphere_joint
- added joint fixed_joint: type fixed, parent auxiliar, child body_link2, origin xyz=0 0 -0.07 rpy=0 0 0
- joint continuous_joint: origin xyz=0 0 0 rpy=0 0 0 -> xyz=0 0 0 rpy=1.55 0 0; parent  -> back_sphere

File: URDFs_set/B_joint_continuous_LEFT.urdf (robot description, URDF)
Before this commit: robot L_JOINT_CONTI, 1 links, 2 joints
Links:
- link auxiliar: geometry collision sphere radius=0.05; visual cylinder length=0.07 radius=0.05
Joints:
- removed joint front_sphere_joint
- added joint fixed_joint: type fixed, parent auxiliar, child body_link2, origin xyz=0 0 -0.07 rpy=0 0 0
- joint continuous_joint: origin xyz=0 0 0 rpy=0 0 0 -> xyz=0 0 0 rpy=0 1.55 0; parent  -> back_sphere

File: URDFs_set/B_joint_continuous_TOP.urdf (robot description, URDF)
Before this commit: robot L_JOINT_CONTI, 1 links, 2 joints
Links:
- link auxiliar: geometry collision sphere radius=0.05; visual cylinder length=0.07 radius=0.05
Joints:
- removed joint front_sphere_joint
- added joint fixed_joint: type fixed, parent auxiliar, child body_link2, origin xyz=0 0 0.07 rpy=0 0 0
- joint continuous_joint: parent  -> back_sphere

File: URDFs_set/B_joint_fixed_BACK.urdf (robot description, URDF)
Before this commit: robot L_JOINT_FIX, 1 links, 1 joints
Links:
- link link_square: geometry collision box size=0.07 0.07 0.07; visual box size=0.07 0.07 0.07
Joints:
- joint fixed_joint: origin xyz=0 0.2 0.005 rpy=1.6 0 0 -> xyz=0 -0.07 0 rpy=0 0 0

File: URDFs_set/B_joint_fixed_BOTTOM.urdf (robot description, URDF)
Before this commit: robot L_JOINT_FIX, 1 links, 1 joints
Links:
- link link_square: geometry collision box size=0.07 0.07 0.07; visual box size=0.07 0.07 0.07
Joints:
- joint fixed_joint: origin xyz=0 0.2 0.005 rpy=1.6 0 0 -> xyz=0 0 -0.07 rpy=0 0 0

File: URDFs_set/B_joint_fixed_FRONT.urdf (robot description, URDF)
Before this commit: robot L_JOINT_FIX, 1 links, 1 joints
Links:
- link link_square: geometry collision box size=0.07 0.07 0.07; visual box size=0.07 0.07 0.07
Joints:
- joint fixed_joint: origin xyz=0 0.2 0.005 rpy=1.6 0 0 -> xyz=0 0.07 0 rpy=0 0 0

File: URDFs_set/B_joint_fixed_LEFT.urdf (robot description, URDF)
Before this commit: robot L_JOINT_FIX, 1 links, 1 joints
Links:
- link link_square: geometry collision box size=0.07 0.07 0.07; visual box size=0.07 0.07 0.07
Joints:
- joint fixed_joint: origin xyz=0 0.2 0.005 rpy=1.6 0 0 -> xyz=0.07 0 0 rpy=0 0 0

File: URDFs_set/B_joint_fixed_RIGHT.urdf (robot description, URDF)
Before this commit: robot B_JOINT_fixed, 1 links, 1 joints
Joints:
- joint fixed_joint: child body_link -> ; origin xyz=0 0.1 0 rpy=1.6 0 0 -> xyz=-0.07 0 0 rpy=0 0 0

File: URDFs_set/B_joint_fixed_TOP.urdf (robot description, URDF)
Before this commit: robot L_JOINT_FIX, 1 links, 1 joints
Links:
- link link_square: geometry collision box size=0.07 0.07 0.07; visual box size=0.07 0.07 0.07
Joints:
- joint fixed_joint: origin xyz=0 0.2 0.005 rpy=1.6 0 0 -> xyz=0 0 0.07 rpy=0 0 0

File: URDFs_set/L_joint_revolute.urdf (robot description, URDF)
Before this commit: robot L_JOINT_REVO, 1 links, 2 joints
Joints:
- joint fixed_joint: child limb_joint_bottom_blue_link -> 
- joint revolute_joint: origin xyz=0 0.05 0 rpy=0.05 0 0 -> xyz=0 0 0 rpy=0 0 0; parent body_joint_link -> 

File: URDFs_set/L_joint_revolute_horizontal.urdf (robot description, URDF)
Before this commit: robot L_JOINT_REVO, 1 links, 2 joints
Joints:
- joint fixed_joint: child limb_joint_bottom_blue_link -> 
- joint revolute_joint: origin xyz=0 0.04 0 rpy=-1.5 0 0 -> xyz=0 0 0 rpy=1.5 0 0; parent body_joint_link -> 

File: URDFs_set/limb_Link.urdf (robot description, URDF)
Before this commit: robot Limb_LINK, 2 links, 1 joints
Links:
- added link aux_sphere, mass 0.5; collision sphere radius=0.02; visual sphere radius=0.02
Joints:
- added joint fixed_joint: type fixed, parent aux_sphere, child limb_link, origin xyz=0 0 0.09 rpy=0 0 0
- joint bot_sphere_joint_limb: child limb_link -> limb_joint_bottom_blue_link; parent limb_joint_bottom_blue_link -> limb_link

File: URDFs_set/limb_Link_Small.urdf (robot description, URDF)
Before this commit: robot Link:small, 2 links, 1 joints
Links:
- added link aux_sphere, mass 0.5; collision sphere radius=0.02; visual sphere radius=0.01
Joints:
- added joint fixed_joint: type fixed, parent aux_sphere, child limb_link, origin xyz=0 0 0.045 rpy=0 0 0
- joint bot_sphere_joint_limb: child limb_link -> limb_small_link_robot; parent limb_small_link_robot -> limb_link

File: links_atchmentExample.urdf (robot description, URDF)
Before this commit: robot Limb_LINK, 7 links, 4 joints
Links:
- removed link link_square
- added link auxiliar, mass 0.5; collision sphere radius=0.05; visual cylinder length=0.07 radius=0.05
Joints:
- added joint revolute_joint: type revolute, parent limb_joint_bottom_blue_link2, child auxiliar, origin xyz=0 0 0 rpy=1.5 0 0, axis 0 0 1, limit lower=-1.14 upper=1.14 effort=1.0 velocity=1.0
- joint fixed_joint: child link_square -> limb_joint_bottom_blue_link3; origin xyz=0 0 0.02 rpy=0 0 0 -> xyz=0 0.2 0.005 rpy=1.6 0 0; parent limb_joint_bottom_blue_link2 -> auxiliar

Commit message: Update of joints, links, and new brain format

File: URDFs_set/B_joint_continuous_BACK.urdf (robot description, URDF)
Before this commit: robot B_JOINT_CONTI, 1 links, 2 joints
Links:
- link auxiliar: geometry collision cylinder length=0.07 radius=0.04; visual cylinder length=0.07 radius=0.04

File: URDFs_set/B_joint_continuous_BOTTOM.urdf (robot description, URDF)
Before this commit: robot B_JOINT_CONTI, 1 links, 2 joints
Links:
- link auxiliar: geometry collision cylinder length=0.07 radius=0.04; visual cylinder length=0.07 radius=0.04

File: URDFs_set/B_joint_continuous_FRONT.urdf (robot description, URDF)
Before this commit: robot B_JOINT_CONTI, 1 links, 2 joints
Links:
- link auxiliar: geometry collision cylinder length=0.07 radius=0.04; visual cylinder length=0.07 radius=0.04

File: URDFs_set/B_joint_continuous_LEFT.urdf (robot description, URDF)
Before this commit: robot B_JOINT_CONTI, 1 links, 2 joints
Links:
- link auxiliar: geometry collision cylinder length=0.07 radius=0.04; visual cylinder length=0.07 radius=0.04

File: URDFs_set/B_joint_continuous_RIGHT.urdf (robot description, URDF)
Before this commit: robot B_JOINT_CONTI, 1 links, 2 joints
Links:
- link auxiliar: geometry collision cylinder length=0.07 radius=0.04; visual cylinder length=0.07 radius=0.04

File: URDFs_set/B_joint_continuous_TOP.urdf (robot description, URDF)
Before this commit: robot B_JOINT_CONTI, 1 links, 2 joints
Links:
- link auxiliar: geometry collision cylinder length=0.07 radius=0.04; visual cylinder length=0.07 radius=0.04

File: URDFs_set/B_joint_revolute_BACK.urdf (robot description, URDF)
Before this commit: robot B_JOINT_REVO, 2 links, 3 joints
Links:
- link auxiliar: geometry collision cylinder length=0.07 radius=0.05; visual cylinder length=0.07 radius=0.05

File: URDFs_set/B_joint_revolute_BOTTOM.urdf (robot description, URDF)
Before this commit: robot B_JOINT_REVO, 2 links, 3 joints
Links:
- link auxiliar: geometry collision cylinder length=0.07 radius=0.05; visual cylinder length=0.07 radius=0.05

File: URDFs_set/B_joint_revolute_FRONT.urdf (robot description, URDF)
Before this commit: robot B_JOINT_REVO, 2 links, 3 joints
Links:
- link auxiliar: geometry collision cylinder length=0.07 radius=0.05; visual cylinder length=0.07 radius=0.05

File: URDFs_set/B_joint_revolute_LEFT.urdf (robot description, URDF)
Before this commit: robot B_JOINT_REVO, 2 links, 3 joints
Links:
- link auxiliar: geometry collision cylinder length=0.07 radius=0.05; visual cylinder length=0.07 radius=0.05

File: URDFs_set/B_joint_revolute_RIGHT.urdf (robot description, URDF)
Before this commit: robot B_JOINT_REVO, 2 links, 3 joints
Links:
- link auxiliar: geometry collision cylinder length=0.07 radius=0.05; visual cylinder length=0.07 radius=0.05

File: URDFs_set/B_joint_revolute_TOP.urdf (robot description, URDF)
Before this commit: robot B_JOINT_REVO, 2 links, 3 joints
Links:
- link auxiliar: geometry collision cylinder length=0.07 radius=0.05; visual cylinder length=0.07 radius=0.05

File: URDFs_set/L_joint_continuous.urdf (robot description, URDF)
Before this commit: robot L_JOINT_CONTI, 1 links, 2 joints
Links:
- link auxiliar: geometry collision cylinder length=0.06 radius=0.04; visual cylinder length=0.06 radius=0.04

File: URDFs_set/L_joint_continuous_horizontal.urdf (robot description, URDF)
Before this commit: robot L_JOINT_CONT_HZ, 1 links, 2 joints
Links:
- link auxiliar: geometry collision cylinder length=0.06 radius=0.04; visual cylinder length=0.06 radius=0.04

File: URDFs_set/L_joint_fixed.urdf (robot description, URDF)
Before this commit: robot L_JOINT_FIX, 1 links, 2 joints
Links:
- link link_square: geometry collision box size=0.04 0.04 0.04; visual box size=0.04 0.04 0.04

File: URDFs_set/L_joint_revolute.urdf (robot description, URDF)
Before this commit: robot L_JOINT_REVO, 1 links, 2 joints
Links:
- link auxiliar: geometry collision cylinder length=0.065 radius=0.04; visual cylinder length=0.065 radius=0.04

File: URDFs_set/limb_Link_Small.urdf (robot description, URDF)
Before this commit: robot Link:small, 3 links, 2 joints
Links:
- link : geometry collision sphere radius=0.01; visual sphere radius=0.01
- link limb_link: geometry collision cylinder length=0.10 radius=0.02125; visual box size=0.003 0.003 0.10

Commit message: Joint types corrections
This commit is to correct the type of joint continuous (which does not exist) for revolute to have the same action

File: URDFs_set/B_joint_continuous_BACK.urdf (robot description, URDF)
Before this commit: robot B_JOINT_CONTI, 1 links, 2 joints
Joints:
- joint joint_1: limit (none) -> lower=-1000 upper=1000 effort=1.0 velocity=1.0; type continuous -> revolute

File: URDFs_set/B_joint_continuous_BOTTOM.urdf (robot description, URDF)
Before this commit: robot B_JOINT_CONTI, 1 links, 2 joints
Joints:
- joint joint_1: limit (none) -> lower=-1000 upper=1000 effort=1.0 velocity=1.0; type continuous -> revolute

File: URDFs_set/B_joint_continuous_FRONT.urdf (robot description, URDF)
Before this commit: robot B_JOINT_CONTI, 1 links, 2 joints
Joints:
- joint joint_1: limit (none) -> lower=-1000 upper=1000 effort=1.0 velocity=1.0; type continuous -> revolute

File: URDFs_set/B_joint_continuous_LEFT.urdf (robot description, URDF)
Before this commit: robot B_JOINT_CONTI, 1 links, 2 joints
Joints:
- joint joint_1: limit (none) -> lower=-1000 upper=1000 effort=1.0 velocity=1.0; type continuous -> revolute

File: URDFs_set/B_joint_continuous_RIGHT.urdf (robot description, URDF)
Before this commit: robot B_JOINT_CONTI, 1 links, 2 joints
Joints:
- joint joint_1: limit (none) -> lower=-1000 upper=1000 effort=1.0 velocity=1.0; type continuous -> revolute

File: URDFs_set/B_joint_continuous_TOP.urdf (robot description, URDF)
Before this commit: robot B_JOINT_CONTI, 1 links, 2 joints
Joints:
- joint joint_1: limit (none) -> lower=-1000 upper=1000 effort=1.0 velocity=1.0; type continuous -> revolute

File: URDFs_set/L_joint_continuous.urdf (robot description, URDF)
Before this commit: robot L_JOINT_CONTI, 1 links, 2 joints
Joints:
- joint joint_1: limit (none) -> lower=-1000 upper=1000 effort=1.0 velocity=1.0; type continuous -> revolute

File: URDFs_set/L_joint_continuous_horizontal.urdf (robot description, URDF)
Before this commit: robot L_JOINT_CONT_HZ, 1 links, 2 joints
Joints:
- joint joint_1: limit (none) -> lower=-1000 upper=1000 effort=1.0 velocity=1.0; type continuous -> revolute

File: corrected_robot0.urdf (robot description, URDF)
Before this commit: robot combined_robot0, 16 links, 15 joints
Links:
- link 16 L_joint_revolute: geometry collision cylinder length=0.065 radius=0.04; visual cylinder length=0.065 radius=0.04
- link 2 L_joint_fixed: geometry collision box size=0.04 0.04 0.04; visual box size=0.04 0.04 0.04
- link 4 L_joint_continuous: geometry collision cylinder length=0.06 radius=0.04; visual cylinder length=0.06 radius=0.04
Joints:
- joint joint_5: limit (none) -> lower=-1000 upper=1000 effort=1.0 velocity=1.0; type continuous -> revolute

Commit message: PPO testing and GE

File: URDFs_set/B_joint_continuous_BACK.urdf (robot description, URDF)
Before this commit: robot B_JOINT_CONTI, 1 links, 2 joints
Joints:
- joint joint_1: limit lower=-1000 upper=1000 effort=1.0 velocity=1.0 -> effort=1.0 velocity=1.0; type revolute -> continuous

File: URDFs_set/B_joint_continuous_BOTTOM.urdf (robot description, URDF)
Before this commit: robot B_JOINT_CONTI, 1 links, 2 joints
Joints:
- joint joint_1: limit lower=-1000 upper=1000 effort=1.0 velocity=1.0 -> effort=1.0 velocity=1.0; type revolute -> continuous

File: URDFs_set/B_joint_continuous_FRONT.urdf (robot description, URDF)
Before this commit: robot B_JOINT_CONTI, 1 links, 2 joints
Joints:
- joint joint_1: limit lower=-1000 upper=1000 effort=1.0 velocity=1.0 -> effort=1.0 velocity=1.0; type revolute -> continuous

File: URDFs_set/B_joint_continuous_LEFT.urdf (robot description, URDF)
Before this commit: robot B_JOINT_CONTI, 1 links, 2 joints
Joints:
- joint joint_1: limit lower=-1000 upper=1000 effort=1.0 velocity=1.0 -> effort=1.0 velocity=1.0; type revolute -> continuous

File: URDFs_set/B_joint_continuous_RIGHT.urdf (robot description, URDF)
Before this commit: robot B_JOINT_CONTI, 1 links, 2 joints
Joints:
- joint joint_1: limit lower=-1000 upper=1000 effort=1.0 velocity=1.0 -> effort=1.0 velocity=1.0; type revolute -> continuous

File: URDFs_set/B_joint_continuous_TOP.urdf (robot description, URDF)
Before this commit: robot B_JOINT_CONTI, 1 links, 2 joints
Joints:
- joint joint_1: limit lower=-1000 upper=1000 effort=1.0 velocity=1.0 -> effort=1.0 velocity=1.0; type revolute -> continuous

File: URDFs_set/L_joint_continuous.urdf (robot description, URDF)
Before this commit: robot L_JOINT_CONTI, 1 links, 2 joints
Joints:
- joint joint_1: limit lower=-1000 upper=1000 effort=1.0 velocity=1.0 -> effort=1.0 velocity=1.0; type revolute -> continuous

File: URDFs_set/L_joint_continuous_horizontal.urdf (robot description, URDF)
Before this commit: robot L_JOINT_CONT_HZ, 1 links, 2 joints
Joints:
- joint joint_1: limit lower=-1000 upper=1000 effort=1.0 velocity=1.0 -> effort=1.0 velocity=1.0; type revolute -> continuous

File: URDFs_set/limb_Link_Small.urdf (robot description, URDF)
Before this commit: robot Link:small, 3 links, 2 joints
Links:
- link limb_link: geometry collision cylinder length=0.10 radius=0.02125; visual cylinder length=0.10 radius=0.03
- link limb_small_link_robot: geometry collision sphere radius=0.02125; visual sphere radius=0.03

File: corrected_robot0.urdf (robot description, URDF)
Before this commit: robot combined_robot0, 16 links, 15 joints
Joints:
- joint joint_5: limit lower=-1000 upper=1000 effort=1.0 velocity=1.0 -> effort=1.0 velocity=1.0; type revolute -> continuous

File: corrected_robot1.urdf (robot description, URDF)
Before this commit: robot combined_robot1, 23 links, 22 joints
Links:
- link 18 limb_Link_Small: geometry collision cylinder length=0.10 radius=0.02125; visual cylinder length=0.10 radius=0.03
- link 3 limb_Link_Small: geometry collision cylinder length=0.10 radius=0.02125; visual cylinder length=0.10 radius=0.03
- link extra_sphere_1: geometry collision sphere radius=0.02125; visual sphere radius=0.03
- link extra_sphere_3: geometry collision sphere radius=0.02125; visual sphere radius=0.03
Joints:
- joint joint_1: limit lower=-1000 upper=1000 effort=1.0 velocity=1.0 -> effort=1.0 velocity=1.0; type revolute -> continuous

File: corrected_robot10.urdf (robot description, URDF)
Before this commit: robot combined_robot10, 14 links, 13 joints
Links:
- link 3 limb_Link_Small: geometry collision cylinder length=0.10 radius=0.02125; visual cylinder length=0.10 radius=0.03
- link 5 limb_Link_Small: geometry collision cylinder length=0.10 radius=0.02125; visual cylinder length=0.10 radius=0.03
- link extra_sphere_1: geometry collision sphere radius=0.02125; visual sphere radius=0.03
- link extra_sphere_2: geometry collision sphere radius=0.02125; visual sphere radius=0.03
Joints:
- joint joint_10: limit lower=-1000 upper=1000 effort=1.0 velocity=1.0 -> effort=1.0 velocity=1.0; type revolute -> continuous

File: corrected_robot2.urdf (robot description, URDF)
Before this commit: robot combined_robot2, 26 links, 25 joints
Links:
- link 17 limb_Link_Small: geometry collision cylinder length=0.10 radius=0.02125; visual cylinder length=0.10 radius=0.03
- link extra_sphere_1: geometry collision sphere radius=0.02125; visual sphere radius=0.03
Joints:
- joint joint_19: limit lower=-1000 upper=1000 effort=1.0 velocity=1.0 -> effort=1.0 velocity=1.0; type revolute -> continuous
- joint joint_4: limit lower=-1000 upper=1000 effort=1.0 velocity=1.0 -> effort=1.0 velocity=1.0; type revolute -> continuous
- joint joint_7: limit lower=-1000 upper=1000 effort=1.0 velocity=1.0 -> effort=1.0 velocity=1.0; type revolute -> continuous

File: corrected_robot3.urdf (robot description, URDF)
Before this commit: robot combined_robot3, 9 links, 8 joints
Links:
- link 12 limb_Link_Small: geometry collision cylinder length=0.10 radius=0.02125; visual cylinder length=0.10 radius=0.03
- link extra_sphere_1: geometry collision sphere radius=0.02125; visual sphere radius=0.03
Joints:
- joint joint_4: limit lower=-1000 upper=1000 effort=1.0 velocity=1.0 -> effort=1.0 velocity=1.0; type revolute -> continuous

File: corrected_robot5.urdf (robot description, URDF)
Before this commit: robot combined_robot5, 12 links, 11 joints
Joints:
- joint joint_1: limit lower=-1000 upper=1000 effort=1.0 velocity=1.0 -> effort=1.0 velocity=1.0; type revolute -> continuous
- joint joint_4: limit lower=-1000 upper=1000 effort=1.0 velocity=1.0 -> effort=1.0 velocity=1.0; type revolute -> continuous

File: corrected_robot6.urdf (robot description, URDF)
Before this commit: robot combined_robot6, 9 links, 8 joints
Links:
- link 5 limb_Link_Small: geometry collision cylinder length=0.10 radius=0.02125; visual cylinder length=0.10 radius=0.03
- link extra_sphere_1: geometry collision sphere radius=0.02125; visual sphere radius=0.03
Joints:
- joint joint_1: limit lower=-1000 upper=1000 effort=1.0 velocity=1.0 -> effort=1.0 velocity=1.0; type revolute -> continuous
- joint joint_6: limit lower=-1000 upper=1000 effort=1.0 velocity=1.0 -> effort=1.0 velocity=1.0; type revolute -> continuous

File: corrected_robot7.urdf (robot description, URDF)
Before this commit: robot combined_robot7, 32 links, 31 joints
Links:
- link 28 limb_Link_Small: geometry collision cylinder length=0.10 radius=0.02125; visual cylinder length=0.10 radius=0.03
- link 30 limb_Link_Small: geometry collision cylinder length=0.10 radius=0.02125; visual cylinder length=0.10 radius=0.03
- link extra_sphere_5: geometry collision sphere radius=0.02125; visual sphere radius=0.03
- link extra_sphere_6: geometry collision sphere radius=0.02125; visual sphere radius=0.03
Joints:
- joint joint_13: limit lower=-1000 upper=1000 effort=1.0 velocity=1.0 -> effort=1.0 velocity=1.0; type revolute -> continuous
- joint joint_16: limit lower=-1000 upper=1000 effort=1.0 velocity=1.0 -> effort=1.0 velocity=1.0; type revolute -> continuous
- joint joint_23: limit lower=-1000 upper=1000 effort=1.0 velocity=1.0 -> effort=1.0 velocity=1.0; type revolute -> continuous
- joint joint_5: limit lower=-1000 upper=1000 effort=1.0 velocity=1.0 -> effort=1.0 velocity=1.0; type revolute -> continuous

File: corrected_robot8.urdf (robot description, URDF)
Before this commit: robot combined_robot8, 14 links, 13 joints
Links:
- link 11 limb_Link_Small: geometry collision cylinder length=0.10 radius=0.02125; visual cylinder length=0.10 radius=0.03
- link 15 limb_Link_Small: geometry collision cylinder length=0.10 radius=0.02125; visual cylinder length=0.10 radius=0.03
- link extra_sphere_1: geometry collision sphere radius=0.02125; visual sphere radius=0.03
- link extra_sphere_2: geometry collision sphere radius=0.02125; visual sphere radius=0.03
Joints:
- joint joint_4: limit lower=-1000 upper=1000 effort=1.0 velocity=1.0 -> effort=1.0 velocity=1.0; type revolute -> continuous
- joint joint_9: limit lower=-1000 upper=1000 effort=1.0 velocity=1.0 -> effort=1.0 velocity=1.0; type revolute -> continuous

File: corrected_robot9.urdf (robot description, URDF)
Before this commit: robot combined_robot9, 7 links, 6 joints
Joints:
- joint joint_1: limit lower=-1000 upper=1000 effort=1.0 velocity=1.0 -> effort=1.0 velocity=1.0; type revolute -> continuous
