Commit message: Simetry completed with some changes on urdf set

File: URDFs_set/B_joint_continuous_BACK.urdf (robot description, URDF)
Before this commit: robot B_JOINT_CONTI, 1 links, 2 joints
Joints:
- joint joint_2: origin xyz=0 0 0.035 rpy=0 0 0 -> xyz=0 0 0.035 rpy=-1.55 0 0

File: URDFs_set/B_joint_continuous_FRONT.urdf (robot description, URDF)
Before this commit: robot B_JOINT_CONTI, 1 links, 2 joints
Joints:
- joint joint_2: origin xyz=0 0 -0.035 rpy=0 0 0 -> xyz=0 0 -0.035 rpy=-1.55 0 0

File: URDFs_set/B_joint_continuous_LEFT.urdf (robot description, URDF)
Before this commit: robot B_JOINT_CONTI, 1 links, 2 joints
Joints:
- joint joint_2: origin xyz=0 0 -0.035 rpy=0 0 0 -> xyz=0 0 -0.035 rpy=0 -1.55 0

File: URDFs_set/B_joint_continuous_RIGHT.urdf (robot description, URDF)
Before this commit: robot B_JOINT_CONTI, 1 links, 2 joints
Joints:
- joint joint_2: origin xyz=0 0 0.035 rpy=0 0 0 -> xyz=0 0 0.035 rpy=0 -1.55 0

File: URDFs_set/B_joint_revolute_BOTTOM.urdf (robot description, URDF)
Before this commit: robot B_JOINT_REVO, 2 links, 3 joints
Joints:
- joint joint_3: origin xyz=0 -0.025 0 rpy=0 0 0 -> xyz=0 -0.025 0 rpy=-1.55 0 0

File: URDFs_set/B_joint_revolute_TOP.urdf (robot description, URDF)
Before this commit: robot B_JOINT_REVO, 2 links, 3 joints
Joints:
- joint joint_3: origin xyz=0 0.025 0 rpy=0 0 0 -> xyz=0 0.025 0 rpy=-1.55 0 0

File: URDFs_set/L_joint_fixed.urdf (robot description, URDF)
Before this commit: robot L_JOINT_FIX, 1 links, 2 joints
Joints:
- joint joint_2: origin xyz=0 0 0.01 rpy=0 0 0 -> xyz=0 0 0.012 rpy=0 0 0

File: URDFs_set/L_joint_revolute.urdf (robot description, URDF)
Before this commit: robot L_JOINT_REVO, 1 links, 2 joints
Joints:
- joint joint_2: origin xyz=0 0 0 rpy=-1.55 0 0 -> xyz=0 0.01 0 rpy=-1.55 0 0

File: URDFs_set/simetry.urdf (robot description, URDF)
Before this commit: robot sim, 18 links, 18 joints
Links:
- removed link 1 B_joint_continuous_sim
- removed link 11 B_joint_fixed_sim
- removed link 12 body_Link_CUBE_sim
- removed link 18 B_joint_revolute_sim
- removed link 19 body_Link_CUBE_sim
- removed link 2 body_Link_CUBE_sim
- removed link 25 L_joint_continuous_sim
- removed link 26 limb_Link_sim
- removed link 3 B_joint_continuous_sim
- removed link 4 body_Link_CUBE_sim
- removed link Sphere_1
- removed link Sphere_11
- removed link Sphere_3
- removed link Sphere_5
- removed link Sphere_8
- removed link Sphere_9
- removed link blackSphere_0_sim
- removed link extra_sphere_1_sim
Joints:
- removed joint joint_10
- removed joint joint_11
- removed joint joint_15
- removed joint joint_16
- removed joint joint_17
- removed joint joint_22
- removed joint joint_23
- removed joint joint_24
- removed joint joint_25
- removed joint joint_29
- removed joint joint_3
- removed joint joint_30
- removed joint joint_31
- removed joint joint_34
- removed joint joint_35
- removed joint joint_4
- removed joint joint_5
- removed joint joint_9

File: URDFs_set/symmetry.urdf (robot description, URDF)
Before this commit: robot sim, 18 links, 18 joints
Links:
- removed link 1 B_joint_continuous_sim
- removed link 11 B_joint_fixed_sim
- removed link 12 body_Link_CUBE_sim
- removed link 18 B_joint_revolute_sim
- removed link 19 body_Link_CUBE_sim
- removed link 2 body_Link_CUBE_sim
- removed link 25 L_joint_continuous_sim
- removed link 26 limb_Link_sim
- removed link 3 B_joint_continuous_sim
- removed link 4 body_Link_CUBE_sim
- removed link Sphere_1
- removed link Sphere_11
- removed link Sphere_3
- removed link Sphere_5
- removed link Sphere_8
- removed link blackSphere_0_sim
- removed link extra_sphere_1_sim
- added link 20 B_joint_revolute_sim, mass 0.05; collision cylinder length=0.04 radius=0.02; visual cylinder length=0.04 radius=0.02
- added link 21 body_Link_CUBE_sim, mass 0.1; collision box size=0.046 0.046 0.046; visual box size=0.046 0.046 0.001
- added link Sphere_10, mass 0.004; collision sphere radius=0.01; visual sphere radius=0.01
Joints:
- removed joint joint_10
- removed joint joint_11
- removed joint joint_15
- removed joint joint_16
- removed joint joint_17
- removed joint joint_22
- removed joint joint_23
- removed joint joint_24
- removed joint joint_25
- removed joint joint_29
- removed joint joint_3
- removed joint joint_30
- removed joint joint_31
- removed joint joint_34
- removed joint joint_35
- removed joint joint_4
- removed joint joint_5
- removed joint joint_9
- added joint joint_36: type fixed, parent 18 body_Link_CUBE, child Sphere_9, origin xyz=0 -0.023 0 rpy=0 0 0
- added joint joint_37: type revolute, parent Sphere_9, child 20 B_joint_revolute_sim, origin xyz=0 0 0 rpy=0 0 0, axis 0 0 1, limit lower=-1 upper=1 effort=1.0 velocity=1.0
- added joint joint_38: type fixed, parent 20 B_joint_revolute_sim, child Sphere_10, origin xyz=0 -0.02 0 rpy=0 0 0
- added joint joint_39: type fixed, parent Sphere_10, child 21 body_Link_CUBE_sim, origin xyz=0 -0.025 0 rpy=0 0 0
