Commit message: Teste for autonomous assembly  #2
NOTA -> Ver o porque da construção estar ao contrario / muito pra frente

File: URDFs_set/L_joint_fixed.urdf (robot description, URDF)
Before this commit: robot L_JOINT_FIX, 1 links, 1 joints
Joints:
- added joint fixed_joint_: type fixed, parent , child , origin xyz=0 0.2 0.005 rpy=1.6 0 0
- joint fixed_joint: child  -> link_square; origin xyz=0 0.2 0.005 rpy=1.6 0 0 -> xyz=0 0 0 rpy=0 0 0; parent link_square -> 

File: URDFs_set/limb_Link.urdf (robot description, URDF)
Before this commit: robot Limb_LINK, 3 links, 2 joints
Links:
- removed link aux_sphere
- added link , mass 0.5; collision sphere radius=0.02; visual sphere radius=0.02
Joints:
- removed joint fixed_joint
- added joint fixed_joint_: type fixed, parent aux_sphere, child limb_link, origin xyz=0 0 0.09 rpy=0 0 0

Commit message: Update on URDF set

File: URDFs_set/L_joint_fixed.urdf (robot description, URDF)
Before this commit: robot L_JOINT_FIX, 1 links, 2 joints
Joints:
- joint joint_2: origin xyz=0 0 0 rpy=0 0 0 -> xyz=0 0 0.012 rpy=0 0 0
