Commit message: Update on URDF set

File: URDFs_set/B_joint_revolute_BOTTOM.urdf (robot description, URDF)
Before this commit: robot B_JOINT_REVO, 2 links, 3 joints
Joints:
- joint joint_3: origin xyz=0 -0.025 0 rpy=0 0 0 -> xyz=0 -0.025 0 rpy=1.55 0 0

File: URDFs_set/L_joint_fixed.urdf (robot description, URDF)
Before this commit: robot L_JOINT_FIX, 1 links, 2 joints
Joints:
- joint joint_2: origin xyz=0 0 0.02 rpy=0 0 0 -> xyz=0 0 0.012 rpy=0 0 0
