Commit message: Fitness correction

File: URDFs_set/symmetry.urdf (robot description, URDF)
Before this commit: robot sim, 4 links, 4 joints
Links:
- removed link 20 B_joint_revolute_sim
- removed link 21 body_Link_CUBE_sim
- removed link Sphere_10
- removed link Sphere_9
- added link 5 L_joint_continuous_horizontal_sim, mass 0.05; collision cylinder length=0.04 radius=0.02; visual cylinder length=0.04 radius=0.02
- added link 6 limb_Link_sim, mass 0.05; collision cylinder length=0.0575 radius=0.015; visual cylinder length=0.0575 radius=0.015
- added link Sphere_2, mass 0.004; collision sphere radius=0.01; visual sphere radius=0.01
- added link blackSphere_1_sim, mass 0.004; collision sphere radius=0.01; visual sphere radius=0.01
- added link extra_sphere_2_sim, mass 0.006; collision sphere radius=0.015; visual sphere radius=0.015
Joints:
- removed joint joint_36
- removed joint joint_37
- removed joint joint_38
- removed joint joint_39
- added joint joint_12: type fixed, parent blackSphere_1_sim, child 6 limb_Link_sim, origin xyz=0 0 0.033 rpy=0 0 3.15
- added joint joint_13: type fixed, parent 6 limb_Link_sim, child extra_sphere_2_sim, origin xyz=0 0 0.03 rpy=0 0 0
- added joint joint_7: type fixed, parent 0 body_Link_CUBE, child Sphere_2, origin xyz=0 -0.023 0 rpy=0 0 0
- added joint joint_8: type continuous, parent Sphere_2, child 5 L_joint_continuous_horizontal_sim, origin xyz=0 -0.02 0 rpy=1.55 0 0, axis 0 0 1, limit effort=1.0 velocity=1.0
- added joint joint_9: type fixed, parent 5 L_joint_continuous_horizontal_sim, child blackSphere_1_sim, origin xyz=0.02 0 0.015 rpy=0 1.6 0
