Commit message: Completed and tested code done #1

File: URDFs_set/symmetry.urdf (robot description, URDF)
Before this commit: robot sim, 4 links, 4 joints
Links:
- removed link 1 B_joint_revolute_sim
- removed link 2 body_Link_CUBE_sim
- removed link Sphere_4
- removed link Sphere_5
- added link 2 B_joint_revolute_sim, mass 0.05; collision cylinder length=0.04 radius=0.02; visual cylinder length=0.04 radius=0.02
- added link 3 body_Link_CUBE_sim, mass 0.1; collision box size=0.046 0.046 0.046; visual box size=0.046 0.046 0.046
- added link Sphere_2, mass 0.004; collision sphere radius=0.01; visual sphere radius=0.01
- added link Sphere_3, mass 0.004; collision sphere radius=0.01; visual sphere radius=0.01
Joints:
- removed joint joint_11
- removed joint joint_12
- removed joint joint_13
- removed joint joint_14
- added joint joint_4: type fixed, parent 0 body_Link_CUBE, child Sphere_2, origin xyz=0 -0.023 0 rpy=0 0 0
- added joint joint_5: type revolute, parent Sphere_2, child 2 B_joint_revolute_sim, origin xyz=0 0 0 rpy=0 0 0, axis 0 0 1, limit lower=-1 upper=1 effort=1.0 velocity=1.0
- added joint joint_6: type fixed, parent 2 B_joint_revolute_sim, child Sphere_3, origin xyz=0 -0.02 0 rpy=0 0 0
- added joint joint_7: type fixed, parent Sphere_3, child 3 body_Link_CUBE_sim, origin xyz=0 -0.025 0 rpy=0 0 0
