Commit message: # 2 Updated joints, links and updated Autonomous_Assembly_working.py

File: Examples of URDF/links_atchmentExample.urdf (robot description, URDF)
Before this commit: robot Link:small, 7 links, 2 joints
Links:
- removed link link_square
- added link auxiliar, mass 0.5; collision cylinder length=0.07 radius=0.03; visual cylinder length=0.07 radius=0.04

File: URDFs_set/B_joint_revolute_BACK.urdf (robot description, URDF)
Before this commit: robot B_JOINT_REVO, 2 links, 3 joints
Joints:
- joint joint_1: limit lower=-3.14 upper=3.14 effort=1.0 velocity=1.0 -> lower=-1 upper=1 effort=1.0 velocity=1.0

File: URDFs_set/B_joint_revolute_BOTTOM.urdf (robot description, URDF)
Before this commit: robot B_JOINT_REVO, 2 links, 3 joints
Joints:
- joint joint_1: limit lower=-3.14 upper=3.14 effort=1.0 velocity=1.0 -> lower=-1 upper=1 effort=1.0 velocity=1.0

File: URDFs_set/B_joint_revolute_FRONT.urdf (robot description, URDF)
Before this commit: robot B_JOINT_REVO, 2 links, 3 joints
Joints:
- joint joint_1: limit lower=-3.14 upper=3.14 effort=1.0 velocity=1.0 -> lower=-1 upper=1 effort=1.0 velocity=1.0

File: URDFs_set/B_joint_revolute_LEFT.urdf (robot description, URDF)
Before this commit: robot B_JOINT_REVO, 2 links, 3 joints
Joints:
- joint joint_1: limit lower=-3.14 upper=3.14 effort=1.0 velocity=1.0 -> lower=-1 upper=1 effort=1.0 velocity=1.0

File: URDFs_set/B_joint_revolute_RIGHT.urdf (robot description, URDF)
Before this commit: robot B_JOINT_REVO, 2 links, 3 joints
Joints:
- joint joint_1: limit lower=-3.14 upper=3.14 effort=1.0 velocity=1.0 -> lower=-1 upper=1 effort=1.0 velocity=1.0

File: URDFs_set/B_joint_revolute_TOP.urdf (robot description, URDF)
Before this commit: robot B_JOINT_REVO, 2 links, 3 joints
Joints:
- joint joint_1: limit lower=-3.14 upper=3.14 effort=1.0 velocity=1.0 -> lower=-1 upper=1 effort=1.0 velocity=1.0

File: URDFs_set/L_joint_continuous.urdf (robot description, URDF)
Before this commit: robot L_JOINT_CONTI, 1 links, 2 joints
Links:
- link auxiliar: geometry collision cylinder length=0.07 radius=0.03; visual cylinder length=0.06 radius=0.04

File: URDFs_set/L_joint_continuous_horizontal.urdf (robot description, URDF)
Before this commit: robot L_JOINT_REVO, 1 links, 2 joints
Links:
- link auxiliar: geometry collision cylinder length=0.07 radius=0.03; visual cylinder length=0.06 radius=0.04
Joints:
- joint joint_1: limit lower=-1.14 upper=1.14 effort=1.0 velocity=1.0 -> (none); origin xyz=0 0 0 rpy=1.5 0 0 -> xyz=0 0 0 rpy=0 0 0; type revolute -> continuous
- joint joint_2: origin xyz=0 0.2 0.005 rpy=1.6 0 0 -> xyz=0.05 0 0 rpy=0 1.6 0

File: URDFs_set/L_joint_fixed.urdf (robot description, URDF)
Before this commit: robot L_JOINT_FIX, 1 links, 2 joints
Links:
- link link_square: geometry collision box size=0.05 0.05 0.05; visual box size=0.04 0.04 0.04

File: URDFs_set/L_joint_revolute.urdf (robot description, URDF)
Before this commit: robot L_JOINT_REVO, 1 links, 2 joints
Links:
- link auxiliar: geometry collision sphere radius=0.05; visual cylinder length=0.065 radius=0.04
Joints:
- joint joint_1: limit lower=-1.14 upper=1.14 effort=1.0 velocity=1.0 -> lower=-0.75 upper=0.75 effort=1.0 velocity=1.0
- joint joint_2: origin xyz=0 0.2 0.005 rpy=1.6 0 0 -> xyz=0 0 0 rpy=0 0 0

File: URDFs_set/limb_Link.urdf (robot description, URDF)
Before this commit: robot Limb_LINK, 3 links, 2 joints
Joints:
- joint joint_1: parent  -> aux_sphere

File: URDFs_set/wheel_link.urdf (robot description, URDF)
Before this commit: robot L_WHEEL, 2 links, 1 joints
Links:
- link : geometry collision sphere length=0.07 radius=0.05; visual cylinder length=0.1 radius=0.01
- link limb_link: geometry collision cylinder length=0.025 radius=0.07; visual cylinder length=0.025 radius=0.07
Joints:
- joint joint_1: child wheel_link -> limb_link; origin xyz=0 0 0 rpy=0 0 0 -> xyz=0 0 0.04 rpy=0 0 0; parent  -> a

File: corrected_robot0.urdf (robot description, URDF)
Before this commit: robot combined_robot0, 14 links, 3 joints
Links:
- link 2 L_joint_continuous: geometry collision cylinder length=0.07 radius=0.03; visual cylinder length=0.06 radius=0.04
- link 5 L_joint_fixed: geometry collision box size=0.05 0.05 0.05; visual box size=0.04 0.04 0.04
- link 6 wheel_link: geometry collision cylinder length=0.025 radius=0.07; visual cylinder length=0.025 radius=0.07
- link blackSphere_1: geometry collision sphere length=0.07 radius=0.05; visual cylinder length=0.1 radius=0.01
Joints:
- joint joint_1: limit lower=-3.14 upper=3.14 effort=1.0 velocity=1.0 -> lower=-1 upper=1 effort=1.0 velocity=1.0
