Commit message: Update of joints' names and autonomous assembly

File: Examples of URDF/URDF_TESTING.urdf (robot description, URDF)
Before this commit: robot BODY_LINK, 4 links, 3 joints
Links:
- added link bottom_sphere, mass 0.5; collision sphere radius=0.02; visual sphere radius=0.02
Joints:
- removed joint continuous_joint
- added joint cube2_connection_joint: type fixed, parent bottom_sphere, child body_link2, origin xyz=0 -0.05 0 rpy=0 0 0
- added joint revolute_joint: type revolute, parent back_sphere, child auxiliar, origin xyz=0 0 0 rpy=0 0 0, axis 0 0 1, limit lower=-3.14 upper=3.14 effort=1.0 velocity=1.0
- joint back_sphere_joint: origin xyz=0.05 0 0 rpy=0 1.55 0 -> xyz=0 -0.05 0 rpy=0 1.55 0
- joint fixed_joint: child body_link2 -> bottom_sphere; origin xyz=0 0 0.07 rpy=0 0 0 -> xyz=0 -0.05 0 rpy=0 0 0

File: URDFs_set/B_joint_continuous_BACK.urdf (robot description, URDF)
Before this commit: robot B_JOINT_CONTI, 1 links, 2 joints
Joints:
- removed joint continuous_joint
- removed joint fixed_joint
- added joint joint_1: type continuous, parent back_sphere, child auxiliar, origin xyz=0 0 0 rpy=1.55 0 0, axis 0 0 1
- added joint joint_2: type fixed, parent auxiliar, child body_link2, origin xyz=0 0 0.07 rpy=0 0 0

File: URDFs_set/B_joint_continuous_BOTTOM.urdf (robot description, URDF)
Before this commit: robot B_JOINT_CONTI, 1 links, 2 joints
Joints:
- removed joint continuous_joint
- removed joint fixed_joint
- added joint joint_1: type continuous, parent back_sphere, child auxiliar, origin xyz=0 0 0 rpy=0 0 0, axis 0 0 1
- added joint joint_2: type fixed, parent auxiliar, child body_link2, origin xyz=0 0 -0.07 rpy=0 0 0

File: URDFs_set/B_joint_continuous_FRONT.urdf (robot description, URDF)
Before this commit: robot B_JOINT_CONTI, 1 links, 2 joints
Joints:
- removed joint continuous_joint
- removed joint fixed_joint
- added joint joint_1: type continuous, parent back_sphere, child auxiliar, origin xyz=0 0 0 rpy=1.55 0 0, axis 0 0 1
- added joint joint_2: type fixed, parent auxiliar, child body_link2, origin xyz=0 0 -0.07 rpy=0 0 0

File: URDFs_set/B_joint_continuous_LEFT.urdf (robot description, URDF)
Before this commit: robot B_JOINT_CONTI, 1 links, 2 joints
Joints:
- removed joint continuous_joint
- removed joint fixed_joint
- added joint joint_1: type continuous, parent back_sphere, child auxiliar, origin xyz=0 0 0 rpy=0 1.55 0, axis 0 0 1
- added joint joint_2: type fixed, parent auxiliar, child body_link2, origin xyz=0 0 -0.07 rpy=0 0 0

File: URDFs_set/B_joint_continuous_RIGHT.urdf (robot description, URDF)
Before this commit: robot B_JOINT_CONTI, 1 links, 2 joints
Joints:
- removed joint continuous_joint
- removed joint fixed_joint
- added joint joint_1: type continuous, parent back_sphere, child auxiliar, origin xyz=0 0 0 rpy=0 1.55 0, axis 0 0 1
- added joint joint_2: type fixed, parent auxiliar, child body_link2, origin xyz=0 0 0.07 rpy=0 0 0

File: URDFs_set/B_joint_continuous_TOP.urdf (robot description, URDF)
Before this commit: robot B_JOINT_CONTI, 1 links, 2 joints
Joints:
- removed joint continuous_joint
- removed joint fixed_joint
- added joint joint_1: type continuous, parent back_sphere, child auxiliar, origin xyz=0 0 0 rpy=0 0 0, axis 0 0 1
- added joint joint_2: type fixed, parent auxiliar, child body_link2, origin xyz=0 0 0.07 rpy=0 0 0

File: URDFs_set/B_joint_fixed_BACK.urdf (robot description, URDF)
Before this commit: robot B_JOINT_fixed, 1 links, 2 joints
Joints:
- removed joint fixed_joint
- removed joint fixed_joint_
- added joint joint_1: type fixed, parent , child link_square, origin xyz=0 0 0 rpy=0 0 0
- added joint joint_2: type fixed, parent link_square, child , origin xyz=0 0 0 rpy=0 0 0

File: URDFs_set/B_joint_fixed_BOTTOM.urdf (robot description, URDF)
Before this commit: robot B_JOINT_fixed, 1 links, 1 joints
Joints:
- removed joint fixed_joint
- added joint joint_1: type fixed, parent , child link_square, origin xyz=0 0 0 rpy=0 0 0
- added joint joint_2: type fixed, parent link_square, child , origin xyz=0 0 -0.07 rpy=0 0 0

File: URDFs_set/B_joint_fixed_FRONT.urdf (robot description, URDF)
Before this commit: robot B_JOINT_fixed, 1 links, 1 joints
Joints:
- removed joint fixed_joint
- added joint joint_1: type fixed, parent , child link_square, origin xyz=0 0 0 rpy=0 0 0
- added joint joint_2: type fixed, parent link_square, child , origin xyz=0 0.07 0 rpy=0 0 0

File: URDFs_set/B_joint_fixed_LEFT.urdf (robot description, URDF)
Before this commit: robot B_JOINT_fixed, 1 links, 1 joints
Joints:
- removed joint fixed_joint
- added joint joint_1: type fixed, parent , child link_square, origin xyz=0 0 0 rpy=0 0 0
- added joint joint_2: type fixed, parent link_square, child , origin xyz=0.07 0 0 rpy=0 0 0

File: URDFs_set/B_joint_fixed_RIGHT.urdf (robot description, URDF)
Before this commit: robot B_JOINT_fixed, 1 links, 1 joints
Joints:
- removed joint fixed_joint
- added joint joint_1: type fixed, parent , child link_square, origin xyz=0 0 0 rpy=0 0 0
- added joint joint_2: type fixed, parent link_square, child , origin xyz=-0.07 0 0 rpy=0 0 0

File: URDFs_set/B_joint_fixed_TOP.urdf (robot description, URDF)
Before this commit: robot B_JOINT_fixed, 1 links, 1 joints
Joints:
- removed joint fixed_joint
- added joint joint_1: type fixed, parent , child link_square, origin xyz=0 0 0 rpy=0 0 0
- added joint joint_2: type fixed, parent link_square, child , origin xyz=0 0 0.07 rpy=0 0 0

File: URDFs_set/B_joint_revolute_BOTTOM.urdf (robot description, URDF)
Before this commit: robot B_JOINT_REVO, 2 links, 3 joints
Joints:
- removed joint connection_joint
- removed joint fixed_joint
- removed joint revolute_joint
- added joint joint_1: type revolute, parent , child auxiliar, origin xyz=0 0 0 rpy=1.55 0 0, axis 0 0 1, limit lower=-3.14 upper=3.14 effort=1.0 velocity=1.0
- added joint joint_2: type fixed, parent auxiliar, child bottom_sphere, origin xyz=0 -0.05 0 rpy=0 0 0
- added joint joint_3: type fixed, parent bottom_sphere, child , origin xyz=0 -0.05 0 rpy=0 0 0

File: URDFs_set/B_joint_revolute_LEFT.urdf (robot description, URDF)
Before this commit: robot B_JOINT_REVO, 2 links, 3 joints
Joints:
- removed joint connection_joint
- removed joint fixed_joint
- removed joint revolute_joint
- added joint joint_1: type revolute, parent , child auxiliar, origin xyz=0 0 0 rpy=0 0 0, axis 0 0 1, limit lower=-3.14 upper=3.14 effort=1.0 velocity=1.0
- added joint joint_2: type fixed, parent auxiliar, child bottom_sphere, origin xyz=-0.05 0 0 rpy=0 0 0
- added joint joint_3: type fixed, parent bottom_sphere, child , origin xyz=-0.05 0 0 rpy=0 0 0

File: URDFs_set/B_joint_revolute_RIGHT.urdf (robot description, URDF)
Before this commit: robot B_JOINT_REVO, 2 links, 3 joints
Joints:
- removed joint cube2_connection_joint
- removed joint fixed_joint
- removed joint revolute_joint
- added joint joint_1: type revolute, parent , child auxiliar, origin xyz=0 0 0 rpy=0 0 0, axis 0 0 1, limit lower=-3.14 upper=3.14 effort=1.0 velocity=1.0
- added joint joint_2: type fixed, parent auxiliar, child bottom_sphere, origin xyz=0.05 0 0 rpy=0 0 0
- added joint joint_3: type fixed, parent bottom_sphere, child , origin xyz=0.05 0 0 rpy=0 0 0

File: URDFs_set/B_joint_revolute_TOP.urdf (robot description, URDF)
Before this commit: robot B_JOINT_REVO, 2 links, 3 joints
Joints:
- removed joint connection_joint
- removed joint fixed_joint
- removed joint revolute_joint
- added joint joint_1: type revolute, parent , child auxiliar, origin xyz=0 0 0 rpy=1.55 0 0, axis 0 0 1, limit lower=-3.14 upper=3.14 effort=1.0 velocity=1.0
- added joint joint_2: type fixed, parent auxiliar, child bottom_sphere, origin xyz=0 0.05 0 rpy=0 0 0
- added joint joint_3: type fixed, parent bottom_sphere, child , origin xyz=0 0.05 0 rpy=0 0 0

File: URDFs_set/L_joint_continuous.urdf (robot description, URDF)
Before this commit: robot L_JOINT_CONTI, 1 links, 2 joints
Joints:
- removed joint continuous_joint
- removed joint front_sphere_joint
- added joint joint_1: type continuous, parent , child auxiliar, origin xyz=0 0 0 rpy=0 0 0, axis 0 0 1
- added joint joint_12: type fixed, parent auxiliar, child , origin xyz=0 0 -0.04 rpy=0 0 0

File: URDFs_set/L_joint_fixed.urdf (robot description, URDF)
Before this commit: robot L_JOINT_FIX, 1 links, 2 joints
Joints:
- removed joint fixed_joint
- removed joint fixed_joint_
- added joint joint_1: type fixed, parent , child , origin xyz=0 0.2 0.005 rpy=1.6 0 0

File: URDFs_set/L_joint_revolute.urdf (robot description, URDF)
Before this commit: robot L_JOINT_REVO, 1 links, 2 joints
Joints:
- removed joint fixed_joint
- removed joint revolute_joint
- added joint joint_1: type revolute, parent , child auxiliar, origin xyz=0 0 0 rpy=0 0 0, axis 0 0 1, limit lower=-1.14 upper=1.14 effort=1.0 velocity=1.0
- added joint joint_2: type fixed, parent auxiliar, child , origin xyz=0 0.2 0.005 rpy=1.6 0 0
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
Commit message: Updated joints and updated Autonomous_Assembly_working.py

File: Examples of URDF/URDF_TESTING.urdf (robot description, URDF)
Before this commit: robot BODY_LINK, 5 links, 4 joints
Links:
- removed link auxiliar
- removed link bottom_sphere
- added link link_square, mass 1.0; collision box size=0.07 0.07 0.07; visual box size=0.07 0.07 0.07
Joints:
- removed joint back_sphere_joint
- removed joint cube2_connection_joint
- removed joint fixed_joint
- removed joint revolute_joint
- added joint joint_1: type fixed, parent link_square, child body_link2, origin xyz=0 -0.07 0 rpy=0 0 0
- added joint joint_2: type fixed, parent back_sphere, child link_square, origin xyz=0 0 0 rpy=0 0 0

File: Examples of URDF/links_atchmentExample.urdf (robot description, URDF)
Before this commit: robot Limb_LINK, 7 links, 5 joints
Links:
- removed link auxiliar
- removed link limb_joint_bottom_blue_link
- removed link limb_joint_bottom_blue_link2
- removed link limb_joint_bottom_blue_link3
- removed link limb_joint_bottom_blue_link5
- added link aux_sphere, mass 0.5; collision sphere radius=0.02; visual sphere radius=0.01
- added link aux_sphere2, mass 0.5; collision sphere radius=0.02; visual sphere radius=0.01
- added link limb_small_link_robot, mass 2.5; collision sphere radius=0.02125; visual sphere radius=0.02125
- added link limb_small_link_robot2, mass 2.5; collision sphere radius=0.02125; visual sphere radius=0.02125
- added link link_square, mass 1.0; collision box size=0.05 0.05 0.05; visual box size=0.05 0.05 0.05
- link limb_link: geometry collision cylinder length=0.1875 radius=0.02125; visual cylinder length=0.10 radius=0.02125
- link limb_link2: geometry collision cylinder length=0.1875 radius=0.02125; visual cylinder length=0.10 radius=0.02125
Joints:
- removed joint bot_sphere_joint_limb
- removed joint bot_sphere_joint_limb2
- removed joint bot_sphere_joint_limb4
- removed joint fixed_joint
- removed joint revolute_joint
- added joint joint_1: type fixed, parent aux_sphere2, child limb_link2, origin xyz=0 0 0.045 rpy=0 0 0
- added joint joint_2: type fixed, parent limb_link2, child limb_small_link_robot2, origin xyz=0 0 0.05 rpy=0 0 0

File: URDFs_set/B_joint_fixed_BACK.urdf (robot description, URDF)
Before this commit: robot B_JOINT_fixed, 1 links, 2 joints
Joints:
- joint joint_1: child link_square -> ; parent  -> back_sphere
- joint joint_2: child  -> body_link2; origin xyz=0 0 0 rpy=0 0 0 -> xyz=0 -0.07 0 rpy=0 0 0

File: URDFs_set/B_joint_fixed_BOTTOM.urdf (robot description, URDF)
Before this commit: robot B_JOINT_fixed, 1 links, 2 joints
Joints:
- joint joint_1: child link_square -> ; parent  -> back_sphere

File: URDFs_set/B_joint_fixed_FRONT.urdf (robot description, URDF)
Before this commit: robot B_JOINT_fixed, 1 links, 2 joints
Joints:
- joint joint_1: child link_square -> ; parent  -> back_sphere

File: URDFs_set/B_joint_fixed_LEFT.urdf (robot description, URDF)
Before this commit: robot B_JOINT_fixed, 1 links, 2 joints
Joints:
- joint joint_1: child link_square -> ; parent  -> back_sphere

File: URDFs_set/B_joint_fixed_RIGHT.urdf (robot description, URDF)
Before this commit: robot B_JOINT_fixed, 1 links, 2 joints
Joints:
- joint joint_1: child link_square -> ; parent  -> back_sphere

File: URDFs_set/B_joint_fixed_TOP.urdf (robot description, URDF)
Before this commit: robot B_JOINT_fixed, 1 links, 2 joints
Joints:
- joint joint_1: child link_square -> ; parent  -> back_sphere

File: URDFs_set/B_joint_revolute_BOTTOM.urdf (robot description, URDF)
Before this commit: robot B_JOINT_REVO, 2 links, 3 joints
Links:
- removed link bottom_sphere
- added link extra_sphere, mass 0.5; collision sphere radius=0.02; visual sphere radius=0.02

File: URDFs_set/B_joint_revolute_FRONT.urdf (robot description, URDF)
Before this commit: robot B_JOINT_REVO, 2 links, 3 joints
Links:
- removed link bottom_sphere
- added link extra_sphere, mass 0.5; collision sphere radius=0.02; visual sphere radius=0.02

File: URDFs_set/B_joint_revolute_LEFT.urdf (robot description, URDF)
Before this commit: robot B_JOINT_REVO, 2 links, 3 joints
Links:
- removed link bottom_sphere
- added link extra_sphere, mass 0.5; collision sphere radius=0.02; visual sphere radius=0.02

File: URDFs_set/B_joint_revolute_RIGHT.urdf (robot description, URDF)
Before this commit: robot B_JOINT_REVO, 2 links, 3 joints
Links:
- removed link bottom_sphere
- added link extra_sphere, mass 0.5; collision sphere radius=0.02; visual sphere radius=0.02

File: URDFs_set/B_joint_revolute_TOP.urdf (robot description, URDF)
Before this commit: robot B_JOINT_REVO, 2 links, 3 joints
Links:
- removed link bottom_sphere
- added link extra_sphere, mass 0.5; collision sphere radius=0.02; visual sphere radius=0.02

File: URDFs_set/L_joint_continuous.urdf (robot description, URDF)
Before this commit: robot L_JOINT_CONTI, 1 links, 2 joints
Joints:
- joint joint_2: origin xyz=0 0 -0.04 rpy=0 0 0 -> xyz=0 0 0 rpy=0 0 0

File: URDFs_set/L_joint_fixed.urdf (robot description, URDF)
Before this commit: robot L_JOINT_FIX, 1 links, 2 joints
Joints:
- joint joint_2: origin xyz=0 0.2 0.005 rpy=1.6 0 0 -> xyz=0 0 0 rpy=0 0 0

File: URDFs_set/limb_Link.urdf (robot description, URDF)
Before this commit: robot Limb_LINK, 3 links, 2 joints
Joints:
- removed joint bot_sphere_joint_limb
- added joint joint_2: type fixed, parent limb_link, child limb_joint_bottom_blue_link, origin xyz=0 0 0.09 rpy=0 0 0

File: URDFs_set/limb_Link_Small.urdf (robot description, URDF)
Before this commit: robot Link:small, 3 links, 2 joints
Links:
- removed link aux_sphere
- added link , mass 0.5; collision sphere radius=0.02; visual sphere radius=0.01

File: URDFs_set/sphere_auxiliar_Link_BACK.urdf (robot description, URDF)
Before this commit: robot BODY_jointFixed_Back, 1 links, 1 joints
Joints:
- removed joint back_sphere_joint
- added joint joint_1: type fixed, parent , child back_sphere, origin xyz=0 -0.05 0 rpy=0 0 0

File: URDFs_set/wheel_link.urdf (robot description, URDF)
Before this commit: robot L_WHEEL, 2 links, 1 joints
Links:
- removed link wheel_link
- added link limb_link, mass 0.5; collision cylinder length=0.015 radius=0.05; visual cylinder length=0.015 radius=0.06

Commit message: # 3 Updated joints, links and updated Autonomous_Assembly_working.py
New conditions for the placement of the links and joints

File: Examples of URDF/URDF_TESTING.urdf (robot description, URDF)
Before this commit: robot BODY_LINK, 4 links, 2 joints
Links:
- removed link back_sphere
- added link front_sphere, mass 0.5; collision sphere radius=0.02; visual sphere radius=0.02
Joints:
- joint joint_1: child body_link2 -> link_square; origin xyz=0 -0.07 0 rpy=0 0 0 -> xyz=0 0 0 rpy=0 0 0; parent link_square -> front_sphere
- joint joint_2: child link_square -> body_link2; origin xyz=0 0 0 rpy=0 0 0 -> xyz=0 0 0.07 rpy=0 0 0; parent back_sphere -> link_square

File: Examples of URDF/links_atchmentExample.urdf (robot description, URDF)
Before this commit: robot Link:small, 7 links, 2 joints
Links:
- link auxiliar: geometry collision sphere radius=0.05; visual cylinder length=0.065 radius=0.04

File: URDFs_set/B_joint_fixed_LEFT.urdf (robot description, URDF)
Before this commit: robot B_JOINT_fixed, 1 links, 2 joints
Joints:
- joint joint_2: origin xyz=0.07 0 0 rpy=0 0 0 -> xyz=-0.07 0 0 rpy=0 0 0

File: URDFs_set/B_joint_fixed_RIGHT.urdf (robot description, URDF)
Before this commit: robot B_JOINT_fixed, 1 links, 2 joints
Joints:
- joint joint_2: origin xyz=-0.07 0 0 rpy=0 0 0 -> xyz=0.07 0 0 rpy=0 0 0

File: URDFs_set/L_joint_continuous_horizontal.urdf (robot description, URDF)
Before this commit: robot L_JOINT_REVO, 1 links, 2 joints
Joints:
- joint joint_2: origin xyz=0.05 0 0 rpy=0 1.6 0 -> xyz=0.04 0 0.025 rpy=0 1.6 0

File: URDFs_set/L_joint_revolute.urdf (robot description, URDF)
Before this commit: robot L_JOINT_REVO, 1 links, 2 joints
Joints:
- joint joint_2: origin xyz=0 0 0 rpy=0 0 0 -> xyz=0 0 0 rpy=-1.55 0 0

File: URDFs_set/limb_Link.urdf (robot description, URDF)
Before this commit: robot Limb_LINK, 3 links, 2 joints
Links:
- link limb_link: geometry collision cylinder length=0.1875 radius=0.03125; visual box size=0.003 0.003 0.1875
Joints:
- joint joint_1: origin xyz=0 0 0.09 rpy=0 0 0 -> xyz=0 0 0.09 rpy=0 0 3.15

File: URDFs_set/limb_Link_Small.urdf (robot description, URDF)
Before this commit: robot Link:small, 3 links, 2 joints
Links:
- link limb_link: geometry collision cylinder length=0.1875 radius=0.02125; visual box size=0.003 0.003 0.10
Joints:
- joint joint_1: origin xyz=0 0 0.045 rpy=0 0 0 -> xyz=0 0 0.045 rpy=0 0 3.15; parent aux_sphere -> a

File: URDFs_set/wheel_link.urdf (robot description, URDF)
Before this commit: robot L_WHEEL, 2 links, 1 joints
Links:
- link limb_link: geometry collision cylinder length=0.025 radius=0.07; visual box size=0.14 0.004 0.004
