Commit message: Ending PPO Testing and still DSGE changing code

File: Examples of URDF/URDF_TESTING.urdf (robot description, URDF)
Before this commit: robot BODY_LINK, 4 links, 2 joints
Links:
- removed link link_square
- added link auxiliar, mass 0.05; collision cylinder length=0.04 radius=0.02; visual cylinder length=0.04 radius=0.02
- link body_link: mass 5.0 -> 0.1; geometry collision box size=0.046 0.046 0.046; visual box size=0.046 0.046 0.046
- link body_link2: mass 5.0 -> 0.1; geometry collision box size=0.046 0.046 0.046; visual box size=0.046 0.046 0.046
- link front_sphere: geometry collision sphere radius=0.02; visual sphere radius=0.01
Joints:
- joint joint_1: axis (none) -> 0 0 1; child link_square -> auxiliar; limit (none) -> effort=1.0 velocity=1.0; type fixed -> continuous
- joint joint_2: origin xyz=0 0 0.07 rpy=0 0 0 -> xyz=0 0 0.035 rpy=0 0 0; parent link_square -> auxiliar

File: Examples of URDF/links_atchmentExample.urdf (robot description, URDF)
Before this commit: robot Link:small, 7 links, 2 joints
Links:
- removed link limb_link2
- removed link limb_small_link_robot
- removed link limb_small_link_robot2
- added link limb_joint_bottom_blue_link, mass 0.006; collision sphere radius=0.015; visual sphere radius=0.015
- added link limb_joint_bottom_blue_link2, mass 0.006; collision sphere radius=0.015; visual sphere radius=0.015
- added link limb_link10, mass 0.05; collision cylinder length=0.0575 radius=0.015; visual cylinder length=0.0575 radius=0.015
- link aux_sphere: mass 0.5 -> 0.004; geometry collision sphere radius=0.01; visual sphere radius=0.01
- link aux_sphere2: mass 0.5 -> 0.004; geometry collision sphere radius=0.01; visual sphere radius=0.01
- link auxiliar: mass 0.5 -> 0.05; geometry collision cylinder length=0.06 radius=0.04; visual cylinder length=0.04 radius=0.02
- link limb_link: mass 2.5 -> 0.05; geometry collision cylinder length=0.0575 radius=0.015; visual cylinder length=0.0575 radius=0.015
Joints:
- added joint joint_10: type fixed, parent aux_sphere2, child limb_link10, origin xyz=0 0 0.03 rpy=0 0 3.15
- added joint joint_21: type fixed, parent limb_link10, child limb_joint_bottom_blue_link2, origin xyz=0 0 0.03 rpy=0 0 0
- joint joint_1: axis (none) -> 0 0 1; child limb_link2 -> auxiliar; limit (none) -> effort=1.0 velocity=1.0; origin xyz=0 0 0.045 rpy=0 0 0 -> xyz=0 0 0 rpy=0 0 0; parent aux_sphere2 -> limb_joint_bottom_blue_link; type fixed -> revolute
- joint joint_2: child limb_small_link_robot2 -> aux_sphere2; origin xyz=0 0 0.05 rpy=0 0 0 -> xyz=0 0 0 rpy=0 0 0; parent limb_link2 -> auxiliar

File: URDFs_set/B_joint_continuous_BACK.urdf (robot description, URDF)
Before this commit: robot B_JOINT_CONTI, 1 links, 2 joints
Links:
- link auxiliar: mass 0.5 -> 0.05; geometry collision cylinder length=0.04 radius=0.02; visual cylinder length=0.04 radius=0.02
Joints:
- joint joint_2: origin xyz=0 0 0.07 rpy=0 0 0 -> xyz=0 0 0.035 rpy=0 0 0

File: URDFs_set/B_joint_continuous_BOTTOM.urdf (robot description, URDF)
Before this commit: robot B_JOINT_CONTI, 1 links, 2 joints
Links:
- link auxiliar: mass 0.5 -> 0.05; geometry collision cylinder length=0.04 radius=0.02; visual cylinder length=0.04 radius=0.02
Joints:
- joint joint_2: origin xyz=0 0 -0.07 rpy=0 0 0 -> xyz=0 0 -0.035 rpy=0 0 0

File: URDFs_set/B_joint_continuous_FRONT.urdf (robot description, URDF)
Before this commit: robot B_JOINT_CONTI, 1 links, 2 joints
Links:
- link auxiliar: mass 0.5 -> 0.05; geometry collision cylinder length=0.04 radius=0.02; visual cylinder length=0.04 radius=0.02
Joints:
- joint joint_2: origin xyz=0 0 -0.07 rpy=0 0 0 -> xyz=0 0 -0.035 rpy=0 0 0

File: URDFs_set/B_joint_continuous_LEFT.urdf (robot description, URDF)
Before this commit: robot B_JOINT_CONTI, 1 links, 2 joints
Links:
- link auxiliar: mass 0.5 -> 0.05; geometry collision cylinder length=0.04 radius=0.02; visual cylinder length=0.04 radius=0.02
Joints:
- joint joint_2: origin xyz=0 0 -0.07 rpy=0 0 0 -> xyz=0 0 -0.035 rpy=0 0 0

File: URDFs_set/B_joint_continuous_RIGHT.urdf (robot description, URDF)
Before this commit: robot B_JOINT_CONTI, 1 links, 2 joints
Links:
- link auxiliar: mass 0.5 -> 0.05; geometry collision cylinder length=0.04 radius=0.02; visual cylinder length=0.04 radius=0.02
Joints:
- joint joint_2: origin xyz=0 0 0.07 rpy=0 0 0 -> xyz=0 0 0.035 rpy=0 0 0

File: URDFs_set/B_joint_continuous_TOP.urdf (robot description, URDF)
Before this commit: robot B_JOINT_CONTI, 1 links, 2 joints
Links:
- link auxiliar: mass 0.5 -> 0.05; geometry collision cylinder length=0.04 radius=0.02; visual cylinder length=0.04 radius=0.02
Joints:
- joint joint_2: origin xyz=0 0 0.07 rpy=0 0 0 -> xyz=0 0 0.035 rpy=0 0 0

File: URDFs_set/B_joint_fixed_BACK.urdf (robot description, URDF)
Before this commit: robot B_JOINT_fixed, 1 links, 2 joints
Links:
- link link_square: mass 1.0 -> 0.05; geometry collision box size=0.03 0.03 0.03; visual box size=0.03 0.03 0.03
Joints:
- joint joint_2: origin xyz=0 -0.07 0 rpy=0 0 0 -> xyz=0 -0.03 0 rpy=0 0 0

File: URDFs_set/B_joint_fixed_BOTTOM.urdf (robot description, URDF)
Before this commit: robot B_JOINT_fixed, 1 links, 2 joints
Links:
- link link_square: mass 1.0 -> 0.05; geometry collision box size=0.03 0.03 0.03; visual box size=0.03 0.03 0.03
Joints:
- joint joint_2: origin xyz=0 0 -0.07 rpy=0 0 0 -> xyz=0 0 -0.03 rpy=0 0 0

File: URDFs_set/B_joint_fixed_FRONT.urdf (robot description, URDF)
Before this commit: robot B_JOINT_fixed, 1 links, 2 joints
Links:
- link link_square: mass 1.0 -> 0.05; geometry collision box size=0.03 0.03 0.03; visual box size=0.03 0.03 0.03
Joints:
- joint joint_2: origin xyz=0 0.07 0 rpy=0 0 0 -> xyz=0 0.03 0 rpy=0 0 0

File: URDFs_set/B_joint_fixed_LEFT.urdf (robot description, URDF)
Before this commit: robot B_JOINT_fixed, 1 links, 2 joints
Links:
- link link_square: mass 1.0 -> 0.05; geometry collision box size=0.03 0.03 0.03; visual box size=0.03 0.03 0.03
Joints:
- joint joint_2: origin xyz=-0.07 0 0 rpy=0 0 0 -> xyz=-0.03 0 0 rpy=0 0 0

File: URDFs_set/B_joint_fixed_RIGHT.urdf (robot description, URDF)
Before this commit: robot B_JOINT_fixed, 1 links, 2 joints
Links:
- link link_square: mass 1.0 -> 0.05; geometry collision box size=0.03 0.03 0.03; visual box size=0.03 0.03 0.03
Joints:
- joint joint_2: origin xyz=0.07 0 0 rpy=0 0 0 -> xyz=0.03 0 0 rpy=0 0 0

File: URDFs_set/B_joint_fixed_TOP.urdf (robot description, URDF)
Before this commit: robot B_JOINT_fixed, 1 links, 2 joints
Links:
- link link_square: mass 1.0 -> 0.05; geometry collision box size=0.03 0.03 0.03; visual box size=0.03 0.03 0.03
Joints:
- joint joint_2: origin xyz=0 0 0.07 rpy=0 0 0 -> xyz=0 0 0.03 rpy=0 0 0

File: URDFs_set/B_joint_revolute_BACK.urdf (robot description, URDF)
Before this commit: robot B_JOINT_REVO, 2 links, 3 joints
Links:
- link auxiliar: mass 0.5 -> 0.05; geometry collision cylinder length=0.04 radius=0.02; visual cylinder length=0.04 radius=0.02
- link extra_sphere: mass 0.5 -> 0.004; geometry collision sphere radius=0.01; visual sphere radius=0.01
Joints:
- joint joint_2: origin xyz=0 -0.05 0 rpy=0 0 0 -> xyz=0 -0.02 0 rpy=0 0 0
- joint joint_3: origin xyz=0 -0.05 0 rpy=0 0 0 -> xyz=0 -0.025 0 rpy=0 0 0

File: URDFs_set/B_joint_revolute_BOTTOM.urdf (robot description, URDF)
Before this commit: robot B_JOINT_REVO, 2 links, 3 joints
Links:
- link auxiliar: mass 0.5 -> 0.05; geometry collision cylinder length=0.04 radius=0.02; visual cylinder length=0.04 radius=0.02
- link extra_sphere: mass 0.5 -> 0.004; geometry collision sphere radius=0.01; visual sphere radius=0.01
Joints:
- joint joint_2: origin xyz=0 -0.05 0 rpy=0 0 0 -> xyz=0 -0.02 0 rpy=0 0 0
- joint joint_3: origin xyz=0 -0.05 0 rpy=0 0 0 -> xyz=0 -0.025 0 rpy=0 0 0

File: URDFs_set/B_joint_revolute_FRONT.urdf (robot description, URDF)
Before this commit: robot B_JOINT_REVO, 2 links, 3 joints
Links:
- link auxiliar: mass 0.5 -> 0.05; geometry collision cylinder length=0.04 radius=0.02; visual cylinder length=0.04 radius=0.02
- link extra_sphere: mass 0.5 -> 0.004; geometry collision sphere radius=0.01; visual sphere radius=0.01
Joints:
- joint joint_2: origin xyz=0 0.05 0 rpy=0 0 0 -> xyz=0 0.02 0 rpy=0 0 0
- joint joint_3: origin xyz=0 0.05 0 rpy=0 0 0 -> xyz=0 0.025 0 rpy=0 0 0

File: URDFs_set/B_joint_revolute_LEFT.urdf (robot description, URDF)
Before this commit: robot B_JOINT_REVO, 2 links, 3 joints
Links:
- link auxiliar: mass 0.5 -> 0.05; geometry collision cylinder length=0.04 radius=0.02; visual cylinder length=0.04 radius=0.02
- link extra_sphere: mass 0.5 -> 0.004; geometry collision sphere radius=0.01; visual sphere radius=0.01
Joints:
- joint joint_2: origin xyz=-0.05 0 0 rpy=0 0 0 -> xyz=-0.02 0 0 rpy=0 0 0
- joint joint_3: origin xyz=-0.05 0 0 rpy=0 0 0 -> xyz=-0.025 0 0 rpy=0 0 0

File: URDFs_set/B_joint_revolute_RIGHT.urdf (robot description, URDF)
Before this commit: robot B_JOINT_REVO, 2 links, 3 joints
Links:
- link auxiliar: mass 0.5 -> 0.05; geometry collision cylinder length=0.04 radius=0.02; visual cylinder length=0.04 radius=0.02
- link extra_sphere: mass 0.5 -> 0.004; geometry collision sphere radius=0.01; visual sphere radius=0.01
Joints:
- joint joint_2: origin xyz=0.05 0 0 rpy=0 0 0 -> xyz=0.02 0 0 rpy=0 0 0
- joint joint_3: origin xyz=0.05 0 0 rpy=0 0 0 -> xyz=0.025 0 0 rpy=0 0 0

File: URDFs_set/B_joint_revolute_TOP.urdf (robot description, URDF)
Before this commit: robot B_JOINT_REVO, 2 links, 3 joints
Links:
- link auxiliar: mass 0.5 -> 0.05; geometry collision cylinder length=0.04 radius=0.02; visual cylinder length=0.04 radius=0.02
- link extra_sphere: mass 0.5 -> 0.004; geometry collision sphere radius=0.01; visual sphere radius=0.01
Joints:
- joint joint_2: origin xyz=0 0.05 0 rpy=0 0 0 -> xyz=0 0.02 0 rpy=0 0 0
- joint joint_3: origin xyz=0 0.05 0 rpy=0 0 0 -> xyz=0 0.025 0 rpy=0 0 0
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