Commit message: FInal touches on controller part and evolution process

File: robots/robot_0.urdf (robot description, URDF)
Before this commit: robot combined_robot_0, 16 links, 15 joints
Links:
- link blackSphere_1: geometry collision cylinder length=0.04 radius=0.009; visual cylinder length=0.04 radius=0.009
- link blackSphere_2: geometry collision cylinder length=0.04 radius=0.001; visual cylinder length=0.04 radius=0.009
