Commit message: Update to docker

File: robots/robot_GEN_0_number_0.urdf (robot description, URDF)
Before this commit: robot combined_robot_GEN_0_number_0, 22 links, 21 joints
Links:
- removed link 13 L_joint_continuous
- removed link 14 limb_Link
- removed link 15 L_joint_continuous
- removed link 16 limb_Link_Small
- removed link 18 B_joint_fixed
- removed link 19 body_Link_CUBE
- removed link 8 L_joint_continuous_horizontal
- removed link 9 limb_Link
- removed link Sphere_3
- removed link Sphere_4
- removed link blackSphere_0
- removed link blackSphere_1
- removed link blackSphere_2
- removed link extra_sphere_1
- removed link extra_sphere_2
- removed link extra_sphere_3
- added link 12 B_joint_fixed, mass 0.05; collision box size=0.03 0.03 0.03; visual box size=0.03 0.03 0.03
- added link 13 body_Link_CUBE, mass 0.1; collision box size=0.046 0.046 0.046; visual box size=0.046 0.046 0.046
Joints:
- removed joint joint_10
- removed joint joint_11
- removed joint joint_12
- removed joint joint_13
- removed joint joint_14
- removed joint joint_15
- removed joint joint_16
- removed joint joint_17
- removed joint joint_18
- removed joint joint_19
- removed joint joint_20
- removed joint joint_7
- removed joint joint_8
- removed joint joint_9
- joint joint_0: origin xyz=0 0.023 0 rpy=0 0 0 -> xyz=0 0 0.023 rpy=0 0 0
- joint joint_1: origin xyz=0 0 0 rpy=0 0 0 -> xyz=0 0 0 rpy=1.55 0 0
- joint joint_4: origin xyz=0.023 0 0 rpy=0 0 0 -> xyz=0 0.023 0 rpy=0 0 0
- joint joint_5: axis 0 0 1 -> (none); child 8 L_joint_continuous_horizontal -> 12 B_joint_fixed; limit effort=1.0 velocity=1.0 -> (none); origin xyz=0.02 0 0 rpy=0 1.55 0 -> xyz=0 0 0 rpy=0 0 0; type continuous -> fixed
- joint joint_6: child blackSphere_0 -> 13 body_Link_CUBE; origin xyz=0.02 0 0.015 rpy=0 1.6 0 -> xyz=0 0.03 0 rpy=0 0 0; parent 8 L_joint_continuous_horizontal -> 12 B_joint_fixed
