Commit message: Final Update for the controller

File: robots/best_gen_000.urdf (robot description, URDF)
Before this commit: robot combined_robot_GEN_0_number_0, 8 links, 7 joints
Links:
- removed link 1 B_joint_revolute
- removed link 12 B_joint_fixed
- removed link 13 body_Link_CUBE
- removed link Sphere_2
- added link 1 B_joint_continuous, mass 0.05; collision cylinder length=0.04 radius=0.02; visual cylinder length=0.04 radius=0.02
- added link 10 body_Link_CUBE, mass 0.1; collision box size=0.046 0.046 0.046; visual box size=0.046 0.046 0.046
- added link 9 B_joint_fixed, mass 0.05; collision box size=0.03 0.03 0.03; visual box size=0.03 0.03 0.03
Joints:
- removed joint joint_6
- joint joint_0: origin xyz=0 0 0.023 rpy=0 0 0 -> xyz=0 0 -0.023 rpy=0 0 0
- joint joint_1: child 1 B_joint_revolute -> 1 B_joint_continuous; limit lower=-1 upper=1 effort=1.0 velocity=1.0 -> effort=1.0 velocity=1.0; origin xyz=0 0 0 rpy=1.55 0 0 -> xyz=0 0 0 rpy=0 0 0; type revolute -> continuous
- joint joint_2: child Sphere_1 -> 2 body_Link_CUBE; origin xyz=0 0.02 0 rpy=0 0 0 -> xyz=0 0 -0.035 rpy=0 0 0; parent 1 B_joint_revolute -> 1 B_joint_continuous
- joint joint_3: child 2 body_Link_CUBE -> Sphere_1; origin xyz=0 0.025 0 rpy=0 0 0 -> xyz=0 -0.023 0 rpy=0 0 0; parent Sphere_1 -> 0 body_Link_CUBE
- joint joint_4: child Sphere_2 -> 9 B_joint_fixed; origin xyz=0 0.023 0 rpy=0 0 0 -> xyz=0 0 0 rpy=0 0 0; parent 0 body_Link_CUBE -> Sphere_1
- joint joint_5: child 12 B_joint_fixed -> 10 body_Link_CUBE; origin xyz=0 0 0 rpy=0 0 0 -> xyz=0 -0.03 0 rpy=0 0 0; parent Sphere_2 -> 9 B_joint_fixed
